File: Hardware/pcb/pcb v1.brd (EAGLE design)
At the start: 160 x 100 mm, 0 parts

Commit message: Añadir partes y gitignore
Parts:
- added Y1: CFS206, partes:CFS206
Changed lines of the file:
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@@
 <?xml version="1.0" encoding="utf-8"?>
 <!DOCTYPE eagle SYSTEM "eagle.dtd">
-<eagle version="7.5.0">
+<eagle version="7.2.0">
 <drawing>
 <settings>
@@
 <layer number="48" name="Document" color="7" fill="1" visible="yes" active="yes"/>
 <layer number="49" name="Reference" color="7" fill="1" visible="yes" active="yes"/>
+<layer number="50" name="dxf" color="7" fill="1" visible="no" active="no"/>
 <layer number="51" name="tDocu" color="7" fill="1" visible="yes" active="yes"/>
 <layer number="52" name="bDocu" color="7" fill="1" visible="yes" active="yes"/>
+<layer number="53" name="tGND_GNDA" color="7" fill="9" visible="no" active="no"/>
+<layer number="54" name="bGND_GNDA" color="1" fill="9" visible="no" active="no"/>
+<layer number="56" name="wert" color="7" fill="1" visible="no" active="no"/>
+<layer number="57" name="tCAD" color="7" fill="1" visible="no" active="no"/>
 <layer number="90" name="Modules" color="5" fill="1" visible="no" active="no"/>
 <layer number="91" name="Nets" color="2" fill="1" visible="no" active="no"/>
@@
 <layer number="97" name="Info" color="7" fill="1" visible="no" active="no"/>
 <layer number="98" name="Guide" color="6" fill="1" visible="no" active="no"/>
+<layer number="99" name="SpiceOrder" color="7" fill="1" visible="no" active="no"/>
+<layer number="100" name="Muster" color="7" fill="1" visible="no" active="no"/>
+<layer number="101" name="Patch_Top" color="12" fill="4" visible="yes" active="yes"/>
+<layer number="102" name="Vscore" color="7" fill="1" visible="yes" active="yes"/>
+<layer number="103" name="tMap" color="7" fill="1" visible="yes" active="yes"/>
+<layer number="104" name="Name" color="16" fill="1" visible="yes" active="yes"/>
+<layer number="105" name="tPlate" color="7" fill="1" visible="yes" active="yes"/>
+<layer number="106" name="bPlate" color="7" fill="1" visible="yes" active="yes"/>
+<layer number="107" name="Crop" color="7" fill="1" visible="yes" active="yes"/>
+<layer number="108" name="tplace-old" color="10" fill="1" visible="yes" active="yes"/>
+<layer number="109" name="ref-old" color="11" fill="1" visible="yes" active="yes"/>
+<layer number="110" name="fp0" color="7" fill="1" visible="yes" active="yes"/>
+<layer number="111" name="LPC17xx" color="7" fill="1" visible="yes" active="yes"/>
+<layer number="112" name="tSilk" color="7" fill="1" visible="yes" active="yes"/>
+<layer number="113" name="IDFDebug" color="4" fill="1" visible="yes" active="yes"/>
+<layer number="116" name="Patch_BOT" color="9" fill="4" visible="yes" active="yes"/>
+<layer number="121" name="_tsilk" color="7" fill="1" visible="yes" active="yes"/>
+<layer number="122" name="_bsilk" color="7" fill="1" visible="yes" active="yes"/>
+<layer number="123" name="tTestmark" color="7" fill="1" visible="yes" active="yes"/>
+<layer number="124" name="bTestmark" color="7" fill="1" visible="yes" active="yes"/>
+<layer number="125" name="_tNames" color="7" fill="1" visible="yes" active="yes"/>
+<layer number="126" name="_bNames" color="7" fill="1" visible="yes" active="yes"/>
+<layer number="127" name="_tValues" color="7" fill="1" visible="yes" active="yes"/>
+<layer number="128" name="_bValues" color="7" fill="1" visible="yes" active="yes"/>
+<layer number="131" name="tAdjust" color="7" fill="1" visible="yes" active="yes"/>
+<layer number="132" name="bAdjust" color="7" fill="1" visible="yes" active="yes"/>
+<layer number="144" name="Drill_legend" color="7" fill="1" visible="yes" active="yes"/>
+<layer number="150" name="Notes" color="7" fill="1" visible="yes" active="yes"/>
+<layer number="151" name="HeatSink" color="7" fill="1" visible="yes" active="yes"/>
+<layer number="152" name="_bDocu" color="7" fill="1" visible="yes" active="yes"/>
+<layer number="153" name="FabDoc1" color="7" fill="1" visible="yes" active="yes"/>
+<layer number="154" name="FabDoc2" color="7" fill="1" visible="yes" active="yes"/>
+<layer number="155" name="FabDoc3" color="7" fill="1" visible="yes" active="yes"/>
+<layer number="199" name="Contour" color="7" fill="1" visible="yes" active="yes"/>
+<layer number="200" name="200bmp" color="1" fill="10" visible="yes" active="yes"/>
+<layer number="201" name="201bmp" color="2" fill="10" visible="yes" active="yes"/>
+<layer number="202" name="202bmp" color="3" fill="10" visible="yes" active="yes"/>
+<layer number="203" name="203bmp" color="4" fill="10" visible="yes" active="yes"/>
+<layer number="204" name="204bmp" color="5" fill="10" visible="yes" active="yes"/>
+<layer number="205" name="205bmp" color="6" fill="10" visible="yes" active="yes"/>
+<layer number="206" name="206bmp" color="7" fill="10" visible="yes" active="yes"/>
+<layer number="207" name="207bmp" color="8" fill="10" visible="yes" active="yes"/>
+<layer number="208" name="208bmp" color="9" fill="10" visible="yes" active="yes"/>
+<layer number="209" name="209bmp" color="7" fill="1" visible="yes" active="yes"/>
+<layer number="210" name="210bmp" color="7" fill="1" visible="yes" active="yes"/>
+<layer number="211" name="211bmp" color="7" fill="1" visible="yes" active="yes"/>
+<layer number="212" name="212bmp" color="7" fill="1" visible="yes" active="yes"/>
+<layer number="213" name="213bmp" color="7" fill="1" visible="yes" active="yes"/>
+<layer number="214" name="214bmp" color="7" fill="1" visible="yes" active="yes"/>
+<layer number="215" name="215bmp" color="7" fill="1" visible="yes" active="yes"/>
+<layer number="216" name="216bmp" color="7" fill="1" visible="yes" active="yes"/>
+<layer number="217" name="217bmp" color="18" fill="1" visible="no" active="no"/>
+<layer number="218" name="218bmp" color="19" fill="1" visible="no" active="no"/>
+<layer number="219" name="219bmp" color="20" fill="1" visible="no" active="no"/>
+<layer number="220" name="220bmp" color="21" fill="1" visible="no" active="no"/>
+<layer number="221" name="221bmp" color="22" fill="1" visible="no" active="no"/>
+<layer number="222" name="222bmp" color="23" fill="1" visible="no" active="no"/>
+<layer number="223" name="223bmp" color="24" fill="1" visible="no" active="no"/>
+<layer number="224" name="224bmp" color="25" fill="1" visible="no" active="no"/>
+<layer number="248" name="Housing" color="7" fill="1" visible="yes" active="yes"/>
+<layer number="249" name="Edge" color="7" fill="1" visible="yes" active="yes"/>
+<layer number="250" name="Descript" color="3" fill="1" visible="no" active="no"/>
+<layer number="251" name="SMDround" color="12" fill="11" visible="no" active="no"/>
+<layer number="254" name="cooling" color="7" fill="1" visible="yes" active="yes"/>
 </layers>
 <board>
@@
 </autorouter>
 <elements>
+<element name="Y1" library="partes" package="CFS206" value="CFS206" x="1.27" y="-2.54"/>
 </elements>
 <signals>

Commit message: Perifericos agregados
Modulo Grove RFID
RTC
2 Reles
Regulador 3.3v
Buzzer
LED RGB
Parts:
- removed Y1: CFS206, partes:CFS206
- added C1, C2: 1uF, rcl:150CLZ-1010
- added C3, C4: 1uF, rcl:C0805
- added C5, C6, C7: 100nF, rcl:C0805
- added D1, D2: 1N5819HW, diego:SOD-123
- added D3: (no value), SparkFun-LED:WS2812B
- added G1: BATTERY-HOLDER_11.6MM, battery:CELL_RETAINER_11.6MM
- added JP1: M025MM, SparkFun-Connectors:SCREWTERMINAL-5MM-2
- added K1, K2: JS-M1-9V-4, relay:JS-M
- added MDL1: (no value), ESP8266-ESP12E:ESP8266-ESP12E
- added Q1: 32.768kHz 12.5pF, crystal:TC26H
- added Q10, Q3, Q4, Q5, Q6, Q7, Q8, Q9: MOSFET-NCHANNELBSS138, SparkFun-DiscreteSemi:SOT23-3
- added R1, R18, R19, R2, R5, R6, R7, R8, R9: 10k, rcl:R0805
- added R10, R12, R14, R16: 100, rcl:R0805
- added R11, R13, R15, R17: 1M, rcl:R0805
- added RFID1: GROVE-RFID, partes:GROVE-RFID
- added S1: (no value), SparkFun-Electromechanical:SWITCH-SPDT
- added SG1: BUZZERPTH, SparkFun-Electromechanical:BUZZER-12MM
- added U$1: DS1307SO8, SparkFun-FreqCtrl:SO08
- added U1: ADP3338AKCZ-3.3RL7, ADI-Phase-2:SOT230P700X180-4N
- added X1, X2: (no value), con-wago-500:W237-103
Connections:
- new net +3V3: C2.+, C7.1, Q10.1, Q3.1, Q4.1, Q5.1, R19.2, R5.2, R7.2, R8.2, U1.2, U1.4
- new net +5V: C1.+, C3.1, C4.1, C5.1, C6.1, D1.C, D2.C, D3.1, K1.1, K2.1, R1.2, R18.2, R2.2, R6.2, R9.2, RFID1.3, S1.1, SG1.+, U$1.8, U1.3
- new net BUZZER: R16.1, R17.2
- new net GND: C1.-, C2.-, C3.2, C4.2, C5.2, C6.2, C7.2, D3.3, G1.N-, JP1.1, Q6.2, Q7.2, Q8.2, Q9.2, R11.1, R13.1, R15.1, R17.1, U$1.4, U1.1
- new net LED: Q10.2, R19.1
- new net N$1: JP1.2, S1.2
- new net N$11: Q5.3, R9.1, RFID1.1
- new net N$12: D1.A, K1.2, Q7.3
- new net N$13: Q6.1, R10.2
- new net N$14: Q7.1, R12.2
- new net N$15: K1.NC, X1.3
- new net N$16: K1.C, X1.2
- new net N$17: K1.NO, X1.1
- new net N$18: D2.A, K2.2, Q8.3
- new net N$19: Q8.1, R14.2
- new net N$2: Q1.2, U$1.1
- new net N$20: K2.NC, X2.3
- new net N$21: K2.C, X2.2
- new net N$22: K2.NO, X2.1
- new net N$23: Q9.1, R16.2
- new net N$24: Q9.3, SG1.-
- new net N$26: D3.4, Q10.3, R18.1
- new net N$3: Q1.1, U$1.2
- new net N$4: G1.P+@1, G1.P+@2, U$1.3
- new net N$5: Q3.3, R2.1, U$1.6
- new net N$6: R1.1, U$1.7
- new net N$7: Q6.3, RFID1.4
- new net N$9: Q4.3, R6.1, U$1.5
- new net RELE1: R12.1, R13.2
- new net RELE2: R14.1, R15.2
- new net RFIDPW: R10.1, R11.2
- new net RFIDTX33: Q5.2, R8.1
- new net SCL33: Q3.2, R5.1
- new net SDA33: Q4.2, R7.1
Other:
- board size 160 x 100 mm -> 43.2 x 19.1 mm
