File: Hardware/pcb/pcb v1 mod.brd (EAGLE design)
At the start: 43.2 x 19.1 mm, 36 parts, among them K1 JS-M1-9V-4, K2 JS-M1-9V-4, Q1 32.768kHz 12.5pF, Q6 MOSFET-NCHANNELBSS138, Q7 MOSFET-NCHANNELBSS138, Q8 MOSFET-NCHANNELBSS138, Q9 MOSFET-NCHANNELBSS138, U1 ADP3338AKCZ-3.3RL7

Commit message: Quitar el rtc
Parts:
- removed C4: 1uF, rcl:C0805
- removed C5: 100nF, rcl:C0805
- removed G1: BATTERY-HOLDER_11.6MM, battery:CELL_RETAINER_11.6MM
- removed Q1: 32.768kHz 12.5pF, crystal:TC26H
- removed R1: 10k, rcl:R0805
- removed U$1: DS1307SO8, SparkFun-FreqCtrl:SO08
- added JP2: (no value), SparkFun-Connectors:1X04
Connections:
- removed net N$2: Q1.2, U$1.1
- removed net N$3: Q1.1, U$1.2
- removed net N$4: G1.P+@1, G1.P+@2, U$1.3
- removed net N$6: R1.1, U$1.7
- net +5V: now also JP2.2; no longer C4.1, C5.1, R1.2, U$1.8
- net GND: now also JP2.1; no longer C4.2, C5.2, G1.N-, U$1.4
- net SCL5: now also JP2.3; no longer U$1.6
- net SDA5: now also JP2.4; no longer U$1.5
Changed lines of the file:
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@@
 </autorouter>
 <elements>
-<element name="G1" library="battery" package="CELL_RETAINER_11.6MM" value="BATTERY-HOLDER_11.6MM" x="20.32" y="8.89">
-<attribute name="MF" value="KEYSTONE" x="20.32" y="8.89" size="1.778" layer="27" display="off"/>
-<attribute name="MPN" value="2997" x="20.32" y="8.89" size="1.778" layer="27" display="off"/>
-<attribute name="OC_FARNELL" value="2293265" x="20.32" y="8.89" size="1.778" layer="27" display="off"/>
-</element>
-<element name="Q1" library="crystal" package="TC26H" value="32.768kHz 12.5pF" x="8.89" y="5.08">
-<attribute name="MF" value="" x="8.89" y="5.08" size="1.778" layer="27" display="off"/>
-<attribute name="MPN" value="" x="8.89" y="5.08" size="1.778" layer="27" display="off"/>
-<attribute name="OC_NEWARK" value="unknown" x="8.89" y="5.08" size="1.778" layer="27" display="off"/>
-<attribute name="OC_FARNELL" value="unknown" x="8.89" y="5.08" size="1.778" layer="27" display="off"/>
-</element>
 <element name="RFID1" library="partes" package="GROVE-RFID" value="GROVE-RFID" x="-19.05" y="0"/>
 <element name="MDL1" library="ESP8266-ESP12E" package="ESP8266-ESP12E" value="" x="-38.1" y="0"/>
@@
 <attribute name="PROD_ID" value="SWCH-08261" x="-58.42" y="-21.59" size="1.778" layer="27" display="off"/>
 </element>
-<element name="U$1" library="SparkFun-FreqCtrl" package="SO08" value="DS1307SO8" x="-66.04" y="-27.94"/>
-<element name="R1" library="rcl" package="R0805" value="10k" x="-73.66" y="-35.56"/>
 <element name="Q6" library="SparkFun-DiscreteSemi" package="SOT23-3" value="MOSFET-NCHANNELBSS138" x="-77.47" y="-88.9">
 <attribute name="PROD_ID" value="TRANS-00830" x="-77.47" y="-88.9" size="1.778" layer="27" display="off"/>
@@
 <element name="D3" library="SparkFun-LED" package="WS2812B" value="" x="-74.93" y="-209.55"/>
 <element name="C3" library="rcl" package="C0805" value="1uF" x="-76.2" y="-215.9"/>
-<element name="C4" library="rcl" package="C0805" value="1uF" x="-76.2" y="-232.41"/>
-<element name="C5" library="rcl" package="C0805" value="100nF" x="-76.2" y="-238.76"/>
 <element name="C6" library="rcl" package="C0805" value="100nF" x="-76.2" y="-245.11"/>
 <element name="C7" library="rcl" package="C0805" value="100nF" x="-76.2" y="-251.46"/>
+<element name="JP2" library="SparkFun-Connectors" package="1X04" value="" x="-76.2" y="-259.08"/>
 </elements>
 <signals>
@@
 <contactref element="JP1" pad="1"/>
 <contactref element="C2" pad="-"/>
-<contactref element="G1" pad="N-"/>
-<contactref element="U$1" pad="4"/>
 <contactref element="Q6" pad="2"/>
 <contactref element="R11" pad="1"/>
@@
 <contactref element="C3" pad="2"/>
 <contactref element="D3" pad="3"/>
-<contactref element="C4" pad="2"/>
-<contactref element="C5" pad="2"/>
 <contactref element="C6" pad="2"/>
 <contactref element="C7" pad="2"/>
+<contactref element="JP2" pad="1"/>
 <wire x1="-76.52" y1="-181.34" x2="-56.83" y2="-167.64" width="0" layer="19" extent="1-1"/>
 <wire x1="-72.07" y1="-198.12" x2="-76.52" y2="-181.34" width="0" layer="19" extent="1-1"/>
@@
 <wire x1="-72.48" y1="-211.15" x2="-76.52" y2="-205.47" width="0" layer="19" extent="1-1"/>
 <wire x1="-75.25" y1="-215.9" x2="-72.48" y2="-211.15" width="0" layer="19" extent="1-1"/>
-<wire x1="-75.25" y1="-232.41" x2="-75.25" y2="-215.9" width="0" layer="19" extent="1-1"/>
-<wire x1="-75.25" y1="-238.76" x2="-75.25" y2="-232.41" width="0" layer="19" extent="1-1"/>
-<wire x1="-75.25" y1="-245.11" x2="-75.25" y2="-238.76" width="0" layer="19" extent="1-1"/>
+<wire x1="-75.25" y1="-245.11" x2="-75.25" y2="-215.9" width="0" layer="19" extent="1-1"/>
 <wire x1="-75.25" y1="-251.46" x2="-75.25" y2="-245.11" width="0" layer="19" extent="1-1"/>
+<wire x1="-76.2" y1="-259.08" x2="-75.25" y2="-251.46" width="0" layer="19" extent="1-1"/>
 <wire x1="-76.52" y1="-130.54" x2="-56.83" y2="-167.64" width="0" layer="19" extent="1-1"/>
 <wire x1="-72.07" y1="-123.19" x2="-76.52" y2="-130.54" width="0" layer="19" extent="1-1"/>
 <wire x1="-77.15" y1="-100.33" x2="-72.07" y2="-123.19" width="0" layer="19" extent="1-1"/>
 <wire x1="-76.52" y1="-89.9" x2="-77.15" y2="-100.33" width="0" layer="19" extent="1-1"/>
-<wire x1="-64.135" y1="-30.5562" x2="-76.52" y2="-89.9" width="0" layer="19" extent="1-1"/>
-<wire x1="-49.87" y1="-26.67" x2="-64.135" y2="-30.5562" width="0" layer="19" extent="1-1"/>
+<wire x1="-49.87" y1="-26.67" x2="-76.52" y2="-89.9" width="0" layer="19" extent="1-1"/>
 <wire x1="-49.87" y1="-15.24" x2="-49.87" y2="-26.67" width="0" layer="19" extent="1-1"/>
 <wire x1="-48.9204" y1="-0.2286" x2="-49.87" y2="-15.24" width="0" layer="19" extent="1-1"/>
 <wire x1="-34.29" y1="-6.35" x2="-48.9204" y2="-0.2286" width="0" layer="19" extent="1-1"/>
-<wire x1="20.32" y1="8.89" x2="-34.29" y2="-6.35" width="0" layer="19" extent="1-1"/>
 </signal>
 <signal name="+5V">
@@
 <contactref element="C1" pad="+"/>
 <contactref element="S1" pad="1"/>
-<contactref element="U$1" pad="8"/>
-<contactref element="R1" pad="2"/>
 <contactref element="RFID1" pad="3"/>
 <contactref element="D1" pad="C"/>
@@
 <contactref element="C3" pad="1"/>
 <contactref element="C6" pad="1"/>
-<contactref element="C5" pad="1"/>
-<contactref element="C4" pad="1"/>
+<contactref element="JP2" pad="2"/>
 <wire x1="-69.14" y1="-187.96" x2="-70.155" y2="-179.07" width="0" layer="19" extent="1-1"/>
 <wire x1="-77.38" y1="-207.95" x2="-69.14" y2="-187.96" width="0" layer="19" extent="1-1"/>
 <wire x1="-77.15" y1="-215.9" x2="-77.38" y2="-207.95" width="0" layer="19" extent="1-1"/>
-<wire x1="-77.15" y1="-232.41" x2="-77.15" y2="-215.9" width="0" layer="19" extent="1-1"/>
-<wire x1="-77.15" y1="-238.76" x2="-77.15" y2="-232.41" width="0" layer="19" extent="1-1"/>
-<wire x1="-77.15" y1="-245.11" x2="-77.15" y2="-238.76" width="0" layer="19" extent="1-1"/>
+<wire x1="-77.15" y1="-245.11" x2="-77.15" y2="-215.9" width="0" layer="19" extent="1-1"/>
+<wire x1="-73.66" y1="-259.08" x2="-77.15" y2="-245.11" width="0" layer="19" extent="1-1"/>
 <wire x1="-60.61" y1="-150.21" x2="-70.155" y2="-179.07" width="0" layer="19" extent="1-1"/>
 <wire x1="-77.775" y1="-133.35" x2="-60.61" y2="-150.21" width="0" layer="19" extent="1-1"/>
 <wire x1="-60.61" y1="-105.76" x2="-77.775" y2="-133.35" width="0" layer="19" extent="1-1"/>
-<wire x1="-72.71" y1="-35.56" x2="-60.61" y2="-105.76" width="0" layer="19" extent="1-1"/>
-<wire x1="-67.945" y1="-25.3238" x2="-72.71" y2="-35.56" width="0" layer="19" extent="1-1"/>
-<wire x1="-58.42" y1="-19.05" x2="-67.945" y2="-25.3238" width="0" layer="19" extent="1-1"/>
+<wire x1="-58.42" y1="-19.05" x2="-60.61" y2="-105.76" width="0" layer="19" extent="1-1"/>
 <wire x1="-48.9204" y1="-4.8514" x2="-58.42" y2="-19.05" width="0" layer="19" extent="1-1"/>
 <wire x1="-41.57" y1="-15.24" x2="-48.9204" y2="-4.8514" width="0" layer="19" extent="1-1"/>
@@
 <wire x1="-29.29" y1="-6.35" x2="-58.42" y2="-21.59" width="0" layer="19" extent="1-1"/>
 </signal>
-<signal name="N$2">
-<contactref element="Q1" pad="2"/>
-<contactref element="U$1" pad="1"/>
-<wire x1="10.16" y1="5.08" x2="-67.945" y2="-30.5562" width="0" layer="19" extent="1-1"/>
-</signal>
-<signal name="N$3">
-<contactref element="Q1" pad="1"/>
-<contactref element="U$1" pad="2"/>
-<wire x1="7.62" y1="5.08" x2="-66.675" y2="-30.5562" width="0" layer="19" extent="1-1"/>
-</signal>
-<signal name="N$4">
-<contactref element="G1" pad="P+@2"/>
-<contactref element="G1" pad="P+@1"/>
-<contactref element="U$1" pad="3"/>
-<wire x1="13.715" y1="8.89" x2="-65.405" y2="-30.5562" width="0" layer="19" extent="1-1"/>
-<wire x1="26.925" y1="8.89" x2="13.715" y2="8.89" width="0" layer="19" extent="1-1"/>
-</signal>
-<signal name="N$6">
-<contactref element="R1" pad="1"/>
-<contactref element="U$1" pad="7"/>
-<wire x1="-66.675" y1="-25.3238" x2="-74.61" y2="-35.56" width="0" layer="19" extent="1-1"/>
-</signal>
-<signal name="SCL5">
-<contactref element="U$1" pad="6"/>
-</signal>
 <signal name="N$7">
 <contactref element="RFID1" pad="4"/>
@@
 </signal>
 <signal name="SDA5">
-<contactref element="U$1" pad="5"/>
+<contactref element="JP2" pad="4"/>
+</signal>
+<signal name="SCL5">
+<contactref element="JP2" pad="3"/>
 </signal>
 </signals>

Commit message: Modulo reles
Parts:
- removed D1, D2: 1N5819HW, diego:SOD-123
- removed K1, K2: JS-M1-9V-4, relay:JS-M
- removed Q7, Q8: MOSFET-NCHANNELBSS138, SparkFun-DiscreteSemi:SOT23-3
- removed R12, R14: 100, rcl:R0805
- removed R13, R15: 1M, rcl:R0805
- removed X1, X2: (no value), con-wago-500:W237-103
- added JP3: (no value), SparkFun-Connectors:1X04
Connections:
- net RFIDTX5 renamed RFIDTX33
- net SCL5 renamed SCL33
- net SDA5 renamed SDA33
- removed net N$12: D1.A, K1.2, Q7.3
- removed net N$14: Q7.1, R12.2
- removed net N$15: K1.NC, X1.3
- removed net N$16: K1.C, X1.2
- removed net N$17: K1.NO, X1.1
- removed net N$18: D2.A, K2.2, Q8.3
- removed net N$19: Q8.1, R14.2
- removed net N$20: K2.NC, X2.3
- removed net N$21: K2.C, X2.2
- removed net N$22: K2.NO, X2.1
- removed net RELE1: R12.1, R13.2
- removed net RELE2: R14.1, R15.2
- new net RELE1-33: JP3.4
- new net RELE2-33: JP3.3
- net +5V: now also JP3.2; no longer D1.C, D2.C, K1.1, K2.1
- net GND: now also JP3.1; no longer Q7.2, Q8.2, R13.1, R15.1

Commit message: esp y atmega328
Parts:
- removed C3: 1uF, rcl:C0805
- removed C6: 100nF, rcl:C0805
- removed D3: (no value), SparkFun-LED:WS2812B
- added C10, C9: 22pF, rcl:C1206
- added C11, C8: 0.1uF, rcl:C0805
- added D1: LED-RGB-CC-THRUCLEAR, SparkFun-LED:LED-RGB-THRU
- added J3: AVR_SPI_PRG_6PTH, SparkFun-Connectors:2X3
- added JP4, JP5, JP6, JP7: (no value), SparkFun-Connectors:1X03
- added R1, R12, R2, R3, R5, R6, R7: 10k, rcl:R0805
- added R13, R9: 100R, rcl:R0805
- added R4: 100K, rcl:R0805
- added R8: 160R, rcl:R0805
- added U3: ATMEGA328P, SparkFun-DigitalIC:TQFP32-08
- added Y1: 16Mhz, SparkFun-FreqCtrl:HC49US
- moved RFID1 100.3 mm to (75.0, -35.0)
- moved MDL1 49.7 mm to (6.90, 21.0)
Connections:
- net RELE2-33 renamed RELE1
- net RFIDTX33 renamed RFID_TX
- removed net LED5: D3.4
- removed net RELE1-33: JP3.4
- removed net SCL33: JP2.3
- removed net SDA33: JP2.4
- new net ESP_RX_33: JP5.1, JP5.3
- new net ESP_TX_33: JP4.1, JP4.3
- new net N$10: D1.1, R8.2
- new net N$11: C9.1, U3.7, Y1.1
- new net N$12: C10.1, U3.8, Y1.2
- new net N$14: C11.1, U3.20
- new net N$15: D1.3, R9.2
- new net N$16: D1.4, R13.2
- new net N$17: J3.3, U3.17
- new net N$18: J3.1, U3.16
- new net N$19: J3.4, U3.15
- new net N$2: MDL1.3, R5.1
- new net N$20: JP6.2, R12.2
- new net N$3: MDL1.11, R7.1
- new net N$39: J3.5, R4.2, U3.29
- new net N$4: MDL1.12, R12.1
- new net N$5: MDL1.10, R6.2
- new net N$6: JP5.2, MDL1.15
- new net N$8: JP4.2, MDL1.16
- new net N$9: JP7.1, MDL1.1, R3.1
- new net RELE2: JP3.2
- new net SCL: JP2.3, R1.1
- new net SDA: JP2.4, R2.1
- net +3V3: now also JP6.3, MDL1.8, R3.2, R5.2, R7.2
- net +5V: now also C8.1, J3.2, JP3.4, R1.2, R2.2, R4.1, U3.18, U3.4, U3.6; no longer C3.1, C6.1, D3.1, JP3.2
- net GND: now also C10.2, C11.2, C8.2, C9.2, J3.6, JP6.1, JP7.2, MDL1.9, R6.1, U3.21, U3.3, U3.5; no longer C3.2, C6.2, D3.3
Other:
- board size 43.2 x 19.1 mm -> 50 x 50 mm

Commit message: Esquematico completo
Parts:
- removed Q6, Q9: MOSFET-NCHANNELBSS138, SparkFun-DiscreteSemi:SOT23-3
- removed R11, R17: 1M, rcl:R0805
- removed R16: 100, rcl:R0805
- added C3: 1uF, rcl:C1206
- added C4, C5, C6: 100nF, rcl:C0805
- added LVLSHF2: LEVELSHIFTER4, partes:LEVELSHIFTER4
- added Q1: 2N3906, transistor-pnp:TO92
- added R14: 10k, rcl:R0805
- C1: value 1uF -> 10uF; device rcl:150CLZ-1010 -> rcl:E2,5-6
- C11, C8: value 0.1uF -> 100nF
- C2: value 1uF -> 100nF; device rcl:150CLZ-1010 -> rcl:C0805
- C7: value 100nF -> 10uF; device rcl:C0805 -> rcl:E2,5-6
- R10: value 100 -> 10k
- R8: device rcl:R0805 -> rcl:R1206
- moved C1 536.2 mm to (-97.9, -548.9)
- moved C2 531.0 mm to (-98.7, -555.1)
- moved R10 443.3 mm to (-92.0, -537.0)
- moved C7 291.9 mm to (-97.9, -542.5)
- moved D1 12.9 mm to (-78.1, -450.3)
Connections:
- removed net N$13: Q6.1, R10.2
- removed net N$24: Q9.3, SG1.-
- removed net RFIDPW: R10.1, R11.2
- new net LED_B: R13.1, U3.10
- new net LED_G: R9.1, U3.14
- new net LED_R: R8.1, U3.13
- new net N$21: LVLSHF2.HV1, U3.30
- new net N$22: LVLSHF2.HV2, U3.31
- new net RFID_PW: R10.1, U3.9
- net +3V3: now also C1.+, C2.1, C3.1, C4.1, LVLSHF2.LV; no longer C2.+, C7.1
- net +5V: now also C5.1, C6.1, C7.+, LVLSHF2.HV, Q1.3, R14.2; no longer C1.+, RFID1.3, SG1.+
- net BUZZER: now also SG1.+, U3.23; no longer R16.1, R17.2
- net ESP_RX_33: now also LVLSHF2.LV2
- net ESP_TX_33: now also LVLSHF2.LV1
- net GND: now also C2.2, C3.2, C4.2, C5.2, C6.2, C7.-, D1.2, LVLSHF2.GND, LVLSHF2.GND1, RFID1.4, SG1.-; no longer C2.-, C7.2, Q6.2, Q9.2, R11.1, R17.1
- net N$23: now also Q1.1, RFID1.3; no longer Q9.1, R16.2
- net N$7: now also Q1.2, R10.2, R14.1; no longer Q6.3, RFID1.4
- net RELE1: now also U3.24
- net RELE2: now also U3.25
- net RFID_TX: now also U3.32
- net SCL: now also U3.28
- net SDA: now also U3.27
