File: Hardware/pcb/pcb v1 mod/pcb v1 mod.brd (EAGLE design)
At the start: 50 x 50 mm, 42 parts, among them J3 AVR_SPI_PRG_6PTH, Q1 2N3906, U1 ADP3338AKCZ-3.3RL7, U3 ATMEGA328P, Y1 16Mhz

Commit message: Ruteo completo
Parts:
- removed C11: 100nF, rcl:C0805
- removed D1: LED-RGB-CC-THRUCLEAR, SparkFun-LED:LED-RGB-THRU
- removed J3: AVR_SPI_PRG_6PTH, SparkFun-Connectors:2X3
- removed JP6: (no value), SparkFun-Connectors:1X03
- removed LVLSHF2: LEVELSHIFTER4, partes:LEVELSHIFTER4
- removed R14: 10k, rcl:R0805
- removed RFID1: GROVE-RFID, partes:GROVE-RFID
- removed U3: ATMEGA328P, SparkFun-DigitalIC:TQFP32-08
- added J1: AVR_SPI_PRG_6PTH, SparkFun-Connectors:2X3
- added JP8, JP9: M02PTH, SparkFun-Connectors:1X02
- added LED1: 5MMRGBLED, adafruit:LED5MMRGB
- added LVLSHF1: LEVELSHIFTER4, partes:LEVELSHIFTER4
- added R11: 100R, rcl:R0805
- added U2: ATMEGA328P, SparkFun-DigitalIC:TQFP32-08
- C10, C9: value 22pF -> 100nF; device rcl:C1206 -> rcl:C0805
- C2: value 100nF -> 10uF; device rcl:C0805 -> rcl:E2,5-6
- C7: value 10uF -> 22pF; device rcl:E2,5-6 -> rcl:C1206
- C8: value 100nF -> 22pF; device rcl:C0805 -> rcl:C1206
- JP2: device SparkFun-Connectors:1X04 -> SparkFun-Connectors:1X04_NO_SILK
- JP3: device SparkFun-Connectors:1X04 -> SparkFun-Connectors:1X03
- JP4, JP5: device SparkFun-Connectors:1X03 -> SparkFun-Connectors:1X04_NO_SILK
- R10: value 10k -> 160R; device rcl:R0805 -> rcl:R1206
- R12: value 10k -> 100R
- R13: value 100R -> 100K
- R4: value 100K -> 10k
- R8: value 160R -> 10k; device rcl:R1206 -> rcl:R0805
- R9: value 100R -> 10k
- moved C2 605.9 mm to (47.0, 33.0), turned to 270 degrees
- moved C1 599.1 mm to (39.4, 34.3), turned to 270 degrees
- moved C6 599.0 mm to (31.8, 23.5)
- moved Q1 587.3 mm to (24.7, 43.8), turned to 90 degrees
- moved C7 581.3 mm to (20.3, 26.7), flipped to the bottom, turned to 90 degrees
- moved R10 575.5 mm to (10.8, 29.2), turned to 270 degrees
- moved C5 528.0 mm to (31.8, 27.3)
- moved JP5 500.6 mm to (33.0, 38.7), turned to 90 degrees
- moved C4 498.9 mm to (23.5, 6.35), flipped to the bottom
- moved JP4 494.8 mm to (29.2, 38.7), turned to 90 degrees
- moved C3 494.7 mm to (24.1, 8.89), flipped to the bottom
- moved R13 489.9 mm to (50.2, 3.81), turned to 90 degrees
- moved R9 477.0 mm to (9.53, 5.08), flipped to the bottom, turned to 90 degrees
- moved R8 475.2 mm to (13.3, 6.35), flipped to the bottom
- moved JP7 457.2 mm to (33.0, 3.81), turned to 90 degrees
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Connections:
- removed net N$39: J3.5, R4.2, U3.29
- new net AT_RST: J1.5, R13.2, U2.29
- net +3V3: now also C10.1, C2.+, JP3.3, LVLSHF1.LV, R4.2, R8.2, R9.2; no longer C1.+, C2.1, JP6.3, LVLSHF2.LV, R3.2, R5.2, R7.2
- net +5V: now also C1.+, C9.1, J1.2, JP2.4, JP5.2, LVLSHF1.HV, R13.1, R6.2, R7.2, U2.18, U2.4, U2.6; no longer C6.1, C7.+, C8.1, J3.2, JP2.2, JP3.4, LVLSHF2.HV, R1.2, R14.2, R4.1, U3.18, U3.4, U3.6
- net BUZZER: now also U2.23; no longer U3.23
- net ESP_RX_33: now also JP8.1, LVLSHF1.LV2; no longer JP5.1, JP5.3, LVLSHF2.LV2
- net ESP_TX_33: now also JP9.1, LVLSHF1.LV1; no longer JP4.1, JP4.3, LVLSHF2.LV1
- net GND: now also C2.-, C7.2, J1.6, JP4.1, JP5.1, LED1.3, LVLSHF1.GND, LVLSHF1.GND1, R3.1, U2.21, U2.3, U2.5; no longer C11.2, C2.2, C7.-, D1.2, J3.6, JP6.1, LVLSHF2.GND, LVLSHF2.GND1, R6.1, RFID1.4, U3.21, U3.3, U3.5
- net LED_B: now also R12.1, U2.10; no longer R13.1, U3.10
- net LED_G: now also R11.1, U2.14; no longer R9.1, U3.14
- net LED_R: now also R10.1, U2.13; no longer R8.1, U3.13
- net N$10: now also LED1.4, R10.2; no longer D1.1, R8.2
- net N$11: now also C7.1, U2.7; no longer C9.1, U3.7
- net N$12: now also C8.1, U2.8; no longer C10.1, U3.8
- net N$14: now also C6.1, U2.20; no longer C11.1, U3.20
- net N$15: now also LED1.2, R11.2; no longer D1.3, R9.2
- net N$16: now also LED1.1, R12.2; no longer D1.4, R13.2
- net N$17: now also J1.3, U2.17; no longer J3.3, U3.17
- net N$18: now also J1.1, U2.16; no longer J3.1, U3.16
- net N$19: now also J1.4, U2.15; no longer J3.4, U3.15
- net N$2: now also R8.1; no longer R5.1
- net N$20: now also JP3.2, R5.2; no longer JP6.2, R12.2
- net N$21: now also LVLSHF1.HV1, U2.30; no longer LVLSHF2.HV1, U3.30
- net N$22: now also LVLSHF1.HV2, U2.31; no longer LVLSHF2.HV2, U3.31
- net N$23: now also JP4.2; no longer RFID1.3
- net N$3: now also R4.1; no longer R7.1
- net N$4: now also R5.1; no longer R12.1
- net N$5: now also R3.2; no longer R6.2
- net N$6: now also JP8.2; no longer JP5.2
- net N$7: now also R1.2, R2.1; no longer R10.2, R14.1
- net N$8: now also JP9.2; no longer JP4.2
- net N$9: now also R9.1; no longer R3.1
- net RELE1: now also JP2.3, U2.24; no longer JP3.3, U3.24
- net RELE2: now also JP2.2, U2.25; no longer JP3.2, U3.25
- net RFID_PW: now also R1.1, U2.9; no longer R10.1, U3.9
- net RFID_TX: now also JP4.4, U2.32; no longer RFID1.1, U3.32
- net SCL: now also JP5.3, R7.1, U2.28; no longer JP2.3, R1.1, U3.28
- net SDA: now also JP5.4, R6.1, U2.27; no longer JP2.4, R2.1, U3.27
Routing:
- net +5V: track 0.00 -> 252.7 mm, vias 0 -> 11
- net GND: track 0.00 -> 228.8 mm, vias 0 -> 2
- net +3V3: track 0.00 -> 102.2 mm, vias 0 -> 5
- net RFID_TX: track 0.00 -> 84.7 mm, vias 0 -> 1
- net N$1: track 0.00 -> 66.7 mm
- net N$8: track 0.00 -> 52.8 mm, vias 0 -> 2
- net N$19: track 0.00 -> 45.3 mm, vias 0 -> 2
- net N$6: track 0.00 -> 44.2 mm, vias 0 -> 2
- net BUZZER: track 0.00 -> 42.8 mm, vias 0 -> 1
- net SDA: track 0.00 -> 41.8 mm, vias 0 -> 3
- net N$18: track 0.00 -> 39.0 mm, vias 0 -> 2
- net SCL: track 0.00 -> 38.5 mm, vias 0 -> 3
- net N$17: track 0.00 -> 38.3 mm, vias 0 -> 2
- net LED_G: track 0.00 -> 37.2 mm, vias 0 -> 1
- net AT_RST: track 0.00 -> 33.8 mm, vias 0 -> 1
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- added copper zone on layer 16, net +3V3
Other:
- board size 50 x 50 mm -> 60 x 50 mm
- board text added: "+"
- board text added: "-"
- board text added: "5v"
- board text added: "ATMEGA_RST"
- board text added: "AVR_SPI_5v"
- board text added: "B1"
- board text added: "BOOT"
- board text added: "ESP_3.3v"
- board text added: "ESP_RST"
- board text added: "GND"
- board text added: "PRG"
- board text added: "RELE"
- board text added: "RFID"
- board text added: "RL1"
- board text added: "RL2"
- board text added: "RTC"
- board text added: "RX"
- board text added: "SCL"
- board text added: "SDA"
- board text added: "TX"
- board text added: "UnplugBox V1 21-03-16"

Commit message: Correcciones placa
Parts:
- moved JP1 5.08 mm to (53.3, 39.4), turned to 90 degrees
- moved R12 3.61 mm to (9.35, 34.4)
Connections:
- net GND: now also JP1.2; no longer JP1.1
- net N$1: now also JP1.1; no longer JP1.2
Routing:
- net GND: track 228.8 -> 234.5 mm
- net N$16: track 5.77 -> 10.8 mm
- net LED_B: track 28.1 -> 24.2 mm
- net N$14: track 12.9 -> 9.86 mm
- net N$18: track 39.0 -> 38.1 mm
- net N$17: track 38.3 -> 37.4 mm
Other:
- outline, holes or cut-outs redrawn

Commit message: Cambios menores
Parts:
- JP8: value M02PTH -> (none); device SparkFun-Connectors:1X02 -> SparkFun-Connectors:1X03
Connections:
- net GND: now also JP8.3
Routing:
- net +3V3: track 102.2 -> 101.4 mm
- net N$8: track 52.8 -> 52.3 mm
Changed lines of the file:
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@@
 <text x="57.4675" y="44.45" size="1.27" layer="21" font="vector" ratio="12" rot="R90" align="top-center">GND</text>
 <text x="57.4675" y="39.37" size="1.27" layer="21" font="vector" ratio="12" rot="R90" align="top-center">5v</text>
-<text x="41.91" y="3.81" size="0.762" layer="21" font="vector" ratio="12" align="bottom-center">TX</text>
-<text x="37.465" y="3.81" size="0.762" layer="21" font="vector" ratio="12" align="bottom-center">RX</text>
-<text x="40.005" y="2.54" size="0.762" layer="21" font="vector" ratio="12" align="bottom-center">ESP_3.3v</text>
+<text x="44.45" y="6.35" size="0.762" layer="21" font="vector" ratio="12" rot="R90" align="bottom-center">TX</text>
+<text x="40.005" y="6.35" size="0.762" layer="21" font="vector" ratio="12" rot="R90" align="bottom-center">RX</text>
+<text x="39.6875" y="11.43" size="0.762" layer="21" font="vector" ratio="12" rot="R180" align="bottom-center">ESP_3.3v</text>
 <text x="30.48" y="5.08" size="0.762" layer="21" font="vector" ratio="12" rot="R90" align="top-center">ESP_RST</text>
 <text x="48.895" y="4.445" size="0.762" layer="21" font="vector" ratio="12" rot="R90" align="bottom-center">PRG</text>
@@
 <wire x1="35" y1="48.5" x2="35" y2="48" width="0.3048" layer="21"/>
 <wire x1="50.8" y1="7.62" x2="50.8" y2="5.715" width="0.127" layer="21"/>
+<text x="40.005" y="3.81" size="0.762" layer="21" font="vector" ratio="12" rot="R90" align="bottom-center">GND</text>
+<wire x1="36.83" y1="10.795" x2="35.56" y2="10.795" width="0.2032" layer="21"/>
+<wire x1="35.56" y1="10.795" x2="35.56" y2="9.525" width="0.2032" layer="21"/>
+<wire x1="42.2275" y1="10.795" x2="43.815" y2="10.795" width="0.2032" layer="21"/>
+<wire x1="43.815" y1="10.795" x2="43.815" y2="9.525" width="0.2032" layer="21"/>
 </plain>
 <attributes>
@@
 </element>
 <element name="R12" library="rcl" package="R0805" value="100R" x="9.35" y="34.385" smashed="yes" rot="R180">
-<attribute name="NAME" x="10.62" y="36.925" size="1.27" layer="25" font="vector" rot="R180"/>
+<attribute name="NAME" x="11.255" y="36.6075" size="1.27" layer="25" font="vector" rot="R180"/>
 <attribute name="VALUE" x="9.985" y="36.925" size="1.27" layer="27" rot="R180"/>
 </element>
@@
 <attribute name="NAME" x="6.35" y="22.86" size="1.27" layer="21" font="vector" rot="R180"/>
 </element>
-<element name="JP8" library="SparkFun-Connectors" package="1X02" value="M02PTH" x="37.465" y="8.89" smashed="yes" rot="R270">
+<element name="JP8" library="SparkFun-Connectors" package="1X03" value="" x="37.465" y="8.89" smashed="yes" rot="R270">
 <attribute name="VALUE" x="34.29" y="10.16" size="1.27" layer="27" rot="R270"/>
 </element>
@@
 <attribute name="VALUE" x="38.735" y="10.16" size="1.27" layer="27" rot="R270"/>
 </element>
-<element name="JP4" library="SparkFun-Connectors" package="1X04_NO_SILK" value="" x="29.21" y="38.735" rot="R90"/>
+<element name="JP4" library="SparkFun-Connectors" package="1X04_NO_SILK" value="" x="29.21" y="38.735" smashed="yes" rot="R90">
+<attribute name="VALUE" x="32.385" y="37.465" size="1.27" layer="27" rot="R90"/>
+</element>
 </elements>
 <signals>
@@
 <wire x1="19.05" y1="7.305" x2="21.59" y2="7.305" width="0.254" layer="16"/>
 <wire x1="21.59" y1="7.305" x2="22.545" y2="6.35" width="0.254" layer="16"/>
-<wire x1="46.355" y1="3.81" x2="36.83" y2="3.81" width="0.254" layer="16"/>
 <wire x1="36.83" y1="3.81" x2="34.29" y2="6.35" width="0.254" layer="16"/>
 <wire x1="34.29" y1="6.35" x2="33.02" y2="6.35" width="0.254" layer="16"/>
@@
 <wire x1="48.26" y1="44.45" x2="53.26" y2="44.45" width="0.6096" layer="1"/>
 <wire x1="53.26" y1="44.45" x2="53.34" y2="44.37" width="0.6096" layer="1"/>
+<contactref element="JP8" pad="3"/>
+<wire x1="36.83" y1="3.81" x2="37.465" y2="3.81" width="0.254" layer="16"/>
+<wire x1="46.355" y1="3.81" x2="37.465" y2="3.81" width="0.254" layer="16"/>
 </signal>
 <signal name="+5V">
@@
 <wire x1="30.48" y1="6.35" x2="31.75" y2="7.62" width="0.254" layer="16"/>
 <wire x1="31.75" y1="7.62" x2="34.29" y2="7.62" width="0.254" layer="16"/>
-<wire x1="34.29" y1="7.62" x2="37.465" y2="4.445" width="0.254" layer="16"/>
-<wire x1="37.465" y1="4.445" x2="43.815" y2="4.445" width="0.254" layer="16"/>
-<wire x1="43.815" y1="4.445" x2="44.45" y2="5.08" width="0.254" layer="16"/>
-<wire x1="44.45" y1="5.08" x2="44.45" y2="7.62" width="0.254" layer="16"/>
+<wire x1="34.29" y1="7.62" x2="36.83" y2="5.08" width="0.254" layer="16"/>
+<wire x1="36.83" y1="5.08" x2="43.815" y2="5.08" width="0.254" layer="16"/>
+<wire x1="43.815" y1="5.08" x2="44.45" y2="5.715" width="0.254" layer="16"/>
+<wire x1="44.45" y1="5.715" x2="44.45" y2="7.62" width="0.254" layer="16"/>
 <wire x1="44.45" y1="7.62" x2="45.72" y2="8.89" width="0.254" layer="16"/>
 <wire x1="45.72" y1="8.89" x2="46.355" y2="8.89" width="0.254" layer="16"/>
@@
 <wire x1="30.48" y1="8.89" x2="31.75" y2="7.62" width="0.254" layer="1"/>
 <wire x1="31.75" y1="7.62" x2="34.29" y2="7.62" width="0.254" layer="1"/>
-<wire x1="34.29" y1="7.62" x2="37.465" y2="4.445" width="0.254" layer="1"/>
-<wire x1="37.465" y1="4.445" x2="40.005" y2="4.445" width="0.254" layer="1"/>
-<wire x1="40.005" y1="4.445" x2="41.91" y2="6.35" width="0.254" layer="1"/>
+<wire x1="34.29" y1="7.62" x2="36.83" y2="5.08" width="0.254" layer="1"/>
+<wire x1="36.83" y1="5.08" x2="40.64" y2="5.08" width="0.254" layer="1"/>
+<wire x1="40.64" y1="5.08" x2="41.91" y2="6.35" width="0.254" layer="1"/>
 </signal>
 <signal name="ESP_TX_33">

Commit message: Cambio de valores de condensadores
Parts:
- C1: value 10uF -> 1000uF
- C3: value 1uF -> 10uF
Changed lines of the file:
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@@
 <?xml version="1.0" encoding="utf-8"?>
 <!DOCTYPE eagle SYSTEM "eagle.dtd">
-<eagle version="7.4.0">
+<eagle version="7.3.0">
 <drawing>
 <settings>
@@
 <attribute name="VALUE" x="9.985" y="36.925" size="1.27" layer="27" rot="R180"/>
 </element>
-<element name="C3" library="rcl" package="C1206" value="1uF" x="24.13" y="8.89" smashed="yes" rot="MR0">
+<element name="C3" library="rcl" package="C1206" value="10uF" x="24.13" y="8.89" smashed="yes" rot="MR0">
 <attribute name="NAME" x="28.575" y="8.255" size="1.27" layer="26" font="vector" rot="MR0"/>
 <attribute name="VALUE" x="25.4" y="6.35" size="1.27" layer="28" rot="MR0"/>
@@
 </element>
 <element name="R1" library="rcl" package="R0805" value="10k" x="17.78" y="43.18" rot="MR180"/>
-<element name="C1" library="rcl" package="E2,5-6" value="10uF" x="39.37" y="34.29" smashed="yes" rot="R270">
+<element name="C1" library="rcl" package="E2,5-6" value="1000uF" x="39.37" y="34.29" smashed="yes" rot="R270">
 <attribute name="NAME" x="43.053" y="31.496" size="1.27" layer="25" font="vector" ratio="10" rot="R180"/>
 <attribute name="VALUE" x="36.703" y="31.623" size="1.27" layer="27" ratio="10" rot="R270"/>

Commit message: Cambios en algunas resistencias
Parts:
- R13: value 100K -> 10K
- R2: value 10k -> 100k
Changed lines of the file:
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@@
 <element name="C7" library="rcl" package="C1206" value="22pF" x="20.32" y="26.67" rot="MR90"/>
 <element name="C8" library="rcl" package="C1206" value="22pF" x="20.32" y="33.02" rot="MR270"/>
-<element name="R13" library="rcl" package="R0805" value="100K" x="50.165" y="3.81" smashed="yes" rot="R90">
+<element name="R13" library="rcl" package="R0805" value="10K" x="50.165" y="3.81" smashed="yes" rot="R90">
 <attribute name="NAME" x="49.53" y="11.43" size="1.27" layer="25" font="vector" rot="R270"/>
 <attribute name="VALUE" x="52.705" y="3.175" size="1.27" layer="27" rot="R90"/>
@@
 </element>
 <element name="LVLSHF1" library="partes" package="LEVELSHIFTER4" value="LEVELSHIFTER4" x="42.545" y="15.875"/>
-<element name="R2" library="rcl" package="R0805" value="10k" x="19.05" y="46.355" smashed="yes" rot="MR180">
+<element name="R2" library="rcl" package="R0805" value="100k" x="19.05" y="46.355" smashed="yes" rot="MR180">
 <attribute name="NAME" x="20.955" y="46.99" size="1.27" layer="26" font="vector" rot="MR180"/>
 <attribute name="VALUE" x="18.415" y="48.895" size="1.27" layer="28" rot="MR180"/>

Commit message: cambio resistencia led
Parts:
- R10: value 160R -> 100R
Changed lines of the file:
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@@
 <attribute name="VALUE" x="36.195" y="2.54" size="1.27" layer="27" rot="R90"/>
 </element>
-<element name="R10" library="rcl" package="R1206" value="160R" x="10.795" y="29.21" rot="R270"/>
+<element name="R10" library="rcl" package="R1206" value="100R" x="10.795" y="29.21" rot="R270"/>
 <element name="R11" library="rcl" package="R0805" value="100R" x="10.16" y="23.495" smashed="yes" rot="R180">
 <attribute name="NAME" x="11.43" y="22.225" size="1.27" layer="25" font="vector" rot="R180"/>

Commit message: Cambio valor C3
Parts:
- C3: value 10uF -> 100uF
Changed lines of the file:
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@@
 <attribute name="VALUE" x="9.985" y="36.925" size="1.27" layer="27" rot="R180"/>
 </element>
-<element name="C3" library="rcl" package="C1206" value="10uF" x="24.13" y="8.89" smashed="yes" rot="MR0">
+<element name="C3" library="rcl" package="C1206" value="100uF" x="24.13" y="8.89" smashed="yes" rot="MR0">
 <attribute name="NAME" x="28.575" y="8.255" size="1.27" layer="26" font="vector" rot="MR0"/>
 <attribute name="VALUE" x="25.4" y="6.35" size="1.27" layer="28" rot="MR0"/>
