File: Hardware/pcb v2/sch y brd/pcb v2.brd (EAGLE design)
At the start: 160 x 100 mm, 23 parts, among them J1 AVR_SPI_PRG_6PTH, Q1 32.768kHz 12.5pF, Q4 MOSFET-NCHANNELBSS138, U2 ATMEGA328P, Y1 16Mhz

Commit message: pcb v2 buzzer
Parts:
- added C11: 1uF, rcl:C0805
- added Q2: PMBT3904, diego:SOT-23-3
- added R4: 4.7K, rcl:R0805
- added R5: 1K, rcl:R0805
- added SG1: BUZZERPTH, SparkFun-Electromechanical:BUZZER-12MM
Connections:
- net LED_R renamed LED
- removed net LED_B: U2.10
- removed net LED_G: U2.14
- new net N$1: Q2.1, R4.2
- new net N$5: Q2.2, R5.1, SG1.-
- net +5V: now also C11.1, R5.2, SG1.+
- net BUZZER: now also R4.1
- net GND: now also C11.2, Q2.3
Changed lines of the file:
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@@
 <element name="R6" library="rcl" package="R0805" value="10k" x="29.21" y="-144.78"/>
 <element name="C10" library="rcl" package="C0805" value="100nF" x="7.62" y="-144.78"/>
+<element name="SG1" library="SparkFun-Electromechanical" package="BUZZER-12MM" value="BUZZERPTH" x="6.35" y="-160.02"/>
+<element name="Q2" library="diego" package="SOT-23-3" value="PMBT3904" x="-2.54" y="-163.83"/>
+<element name="R4" library="rcl" package="R0805" value="4.7K" x="-1.27" y="-170.18"/>
+<element name="R5" library="rcl" package="R0805" value="1K" x="-1.27" y="-175.26"/>
+<element name="C11" library="rcl" package="C0805" value="1uF" x="-1.27" y="-187.96"/>
 </elements>
 <signals>
@@
 <contactref element="U$1" pad="4"/>
 <contactref element="C10" pad="2"/>
+<contactref element="Q2" pad="3"/>
+<contactref element="C11" pad="2"/>
+<wire x1="-2.54" y1="-162.73" x2="-0.32" y2="-187.96" width="0" layer="19" extent="1-1"/>
+<wire x1="4.445" y1="-148.6662" x2="-2.54" y2="-162.73" width="0" layer="19" extent="1-1"/>
 <wire x1="8.57" y1="-144.78" x2="4.445" y2="-148.6662" width="0" layer="19" extent="1-1"/>
 <wire x1="8.89" y1="-132.08" x2="8.57" y2="-144.78" width="0" layer="19" extent="1-1"/>
@@
 <contactref element="R3" pad="2"/>
 <contactref element="R6" pad="2"/>
-<wire x1="6.67" y1="-144.78" x2="0.635" y2="-143.4338" width="0" layer="19" extent="1-1"/>
+<contactref element="R5" pad="2"/>
+<contactref element="SG1" pad="+"/>
+<contactref element="C11" pad="1"/>
+<wire x1="-0.32" y1="-175.26" x2="-2.22" y2="-187.96" width="0" layer="19" extent="1-1"/>
+<wire x1="9.6" y1="-160.02" x2="-0.32" y2="-175.26" width="0" layer="19" extent="1-1"/>
+<wire x1="6.67" y1="-144.78" x2="9.6" y2="-160.02" width="0" layer="19" extent="1-1"/>
+<wire x1="0.635" y1="-143.4338" x2="6.67" y2="-144.78" width="0" layer="19" extent="1-1"/>
 <wire x1="14.92" y1="-144.78" x2="6.67" y2="-144.78" width="0" layer="19" extent="1-1"/>
 <wire x1="20" y1="-144.78" x2="14.92" y2="-144.78" width="0" layer="19" extent="1-1"/>
@@
 <signal name="BUZZER">
 <contactref element="U2" pad="23"/>
+<contactref element="R4" pad="1"/>
+<wire x1="9.3726" y1="-4.35" x2="-2.22" y2="-170.18" width="0" layer="19" extent="1-1"/>
 </signal>
 <signal name="SDA">
@@
 <contactref element="U2" pad="25"/>
 </signal>
-<signal name="LED_R">
+<signal name="LED">
 <contactref element="U2" pad="13"/>
-</signal>
-<signal name="LED_G">
-<contactref element="U2" pad="14"/>
-</signal>
-<signal name="LED_B">
-<contactref element="U2" pad="10"/>
 </signal>
 <signal name="N$21">
@@
 <wire x1="13.02" y1="-144.78" x2="1.905" y2="-143.4338" width="0" layer="19" extent="1-1"/>
 </signal>
+<signal name="N$1">
+<contactref element="R4" pad="2"/>
+<contactref element="Q2" pad="1"/>
+<wire x1="-3.49" y1="-164.83" x2="-0.32" y2="-170.18" width="0" layer="19" extent="1-1"/>
+</signal>
+<signal name="N$5">
+<contactref element="Q2" pad="2"/>
+<contactref element="R5" pad="1"/>
+<contactref element="SG1" pad="-"/>
+<wire x1="-1.59" y1="-164.83" x2="-2.22" y2="-175.26" width="0" layer="19" extent="1-1"/>
+<wire x1="3.1" y1="-160.02" x2="-1.59" y2="-164.83" width="0" layer="19" extent="1-1"/>
+</signal>
 </signals>

Commit message: pcb v2 rfid
Parts:
- added JP1: (no value), SparkFun-Connectors:1X08
Connections:
- new net +3V3: JP1.8
- new net RFID_INT: JP1.5
- new net RFID_MISO: JP1.4
- new net RFID_MOSI: JP1.3
- new net RFID_RST: JP1.7
- new net RFID_SCK: JP1.2
- new net RFID_SS: JP1.1
- net GND: now also JP1.6
Changed lines of the file:
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@@
 <element name="R5" library="rcl" package="R0805" value="1K" x="-1.27" y="-175.26"/>
 <element name="C11" library="rcl" package="C0805" value="1uF" x="-1.27" y="-187.96"/>
+<element name="JP1" library="SparkFun-Connectors" package="1X08" value="" x="-1.27" y="-195.58"/>
 </elements>
 <signals>
@@
 <contactref element="Q2" pad="3"/>
 <contactref element="C11" pad="2"/>
+<contactref element="JP1" pad="6"/>
+<wire x1="11.43" y1="-195.58" x2="-0.32" y2="-187.96" width="0" layer="19" extent="1-1"/>
 <wire x1="-2.54" y1="-162.73" x2="-0.32" y2="-187.96" width="0" layer="19" extent="1-1"/>
 <wire x1="4.445" y1="-148.6662" x2="-2.54" y2="-162.73" width="0" layer="19" extent="1-1"/>
@@
 <wire x1="3.1" y1="-160.02" x2="-1.59" y2="-164.83" width="0" layer="19" extent="1-1"/>
 </signal>
+<signal name="RFID_MISO">
+<contactref element="JP1" pad="4"/>
+</signal>
+<signal name="RFID_MOSI">
+<contactref element="JP1" pad="3"/>
+</signal>
+<signal name="RFID_SCK">
+<contactref element="JP1" pad="2"/>
+</signal>
+<signal name="RFID_SS">
+<contactref element="JP1" pad="1"/>
+</signal>
+<signal name="RFID_INT">
+<contactref element="JP1" pad="5"/>
+</signal>
+<signal name="RFID_RST">
+<contactref element="JP1" pad="7"/>
+</signal>
+<signal name="+3V3">
+<contactref element="JP1" pad="8"/>
+</signal>
 </signals>

Commit message: libreria AD8192
Parts:
- removed RESET-EN1: (no value), jumper:SJ
- added R7: 0, rcl:R0805
- added U1: AD8192, partes v2:LFCSP56
Connections:
- new net AMUXVCC: U1.47
- new net AVCC: U1.1
- new net AVCC1: U1.10
- new net AVCC2: U1.33
- new net AVCC3: U1.42
- new net AVEE: U1.4
- new net AVEE1: U1.13
- new net AVEE2: U1.30
- new net AVEE3: U1.39
- new net AVEE4: U1.EXP
- new net DVCC: U1.15
- new net DVCC1: U1.21
- new net DVEE: U1.52
- new net N$7: C9.2, R7.2
- new net VTTI: U1.7
- new net VTTI1: U1.36
- new net VTTO: U1.18
- new net VTTO1: U1.24
- net RST_ATM: now also R7.1; no longer C9.2, RESET-EN1.1, RESET-EN1.2
Changed lines of the file:
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@@
 <element name="C2" library="rcl" package="C0805" value="100nF" x="2.54" y="-62.23"/>
 <element name="C3" library="rcl" package="C0805" value="100nF" x="2.54" y="-68.58"/>
-<element name="RESET-EN1" library="jumper" package="SJ" value="" x="2.54" y="-86.36"/>
 <element name="R1" library="rcl" package="R0805" value="1K" x="2.54" y="-96.52"/>
 <element name="C9" library="rcl" package="C0805" value="100nF" x="2.54" y="-102.87"/>
@@
 <element name="C11" library="rcl" package="C0805" value="1uF" x="-1.27" y="-187.96"/>
 <element name="JP1" library="SparkFun-Connectors" package="1X08" value="" x="-1.27" y="-195.58"/>
+<element name="R7" library="rcl" package="R0805" value="0" x="-1.27" y="-200.66"/>
+<element name="U1" library="partes v2" package="LFCSP56" value="AD8192" x="-8.89" y="-196.85"/>
 </elements>
 <signals>
@@
 <contactref element="D2" pad="A"/>
 <contactref element="C1" pad="1"/>
-<contactref element="RESET-EN1" pad="2"/>
-<contactref element="RESET-EN1" pad="1"/>
-<contactref element="C9" pad="2"/>
-<wire x1="3.302" y1="-86.36" x2="3.49" y2="-102.87" width="0" layer="19" extent="1-1"/>
-<wire x1="1.778" y1="-86.36" x2="3.302" y2="-86.36" width="0" layer="19" extent="1-1"/>
-<wire x1="1.59" y1="-55.88" x2="1.778" y2="-86.36" width="0" layer="19" extent="1-1"/>
+<contactref element="R7" pad="1"/>
+<wire x1="1.59" y1="-55.88" x2="-2.22" y2="-200.66" width="0" layer="19" extent="1-1"/>
 <wire x1="4.24" y1="-49.53" x2="1.59" y2="-55.88" width="0" layer="19" extent="1-1"/>
 <wire x1="3.49" y1="-43.18" x2="4.24" y2="-49.53" width="0" layer="19" extent="1-1"/>
@@
 <contactref element="JP1" pad="8"/>
 </signal>
+<signal name="N$7">
+<contactref element="C9" pad="2"/>
+<contactref element="R7" pad="2"/>
+<wire x1="3.49" y1="-102.87" x2="-0.32" y2="-200.66" width="0" layer="19" extent="1-1"/>
+</signal>
+<signal name="AVCC">
+<contactref element="U1" pad="1"/>
+</signal>
+<signal name="AVEE">
+<contactref element="U1" pad="4"/>
+</signal>
+<signal name="VTTI">
+<contactref element="U1" pad="7"/>
+</signal>
+<signal name="AVCC1">
+<contactref element="U1" pad="10"/>
+</signal>
+<signal name="AVEE1">
+<contactref element="U1" pad="13"/>
+</signal>
+<signal name="DVCC">
+<contactref element="U1" pad="15"/>
+</signal>
+<signal name="VTTO">
+<contactref element="U1" pad="18"/>
+</signal>
+<signal name="DVCC1">
+<contactref element="U1" pad="21"/>
+</signal>
+<signal name="VTTO1">
+<contactref element="U1" pad="24"/>
+</signal>
+<signal name="AVEE2">
+<contactref element="U1" pad="30"/>
+</signal>
+<signal name="AVCC2">
+<contactref element="U1" pad="33"/>
+</signal>
+<signal name="VTTI1">
+<contactref element="U1" pad="36"/>
+</signal>
+<signal name="AVEE3">
+<contactref element="U1" pad="39"/>
+</signal>
+<signal name="AVCC3">
+<contactref element="U1" pad="42"/>
+</signal>
+<signal name="AMUXVCC">
+<contactref element="U1" pad="47"/>
+</signal>
+<signal name="DVEE">
+<contactref element="U1" pad="52"/>
+</signal>
+<signal name="AVEE4">
+<contactref element="U1" pad="EXP"/>
+</signal>
 </signals>

Commit message: libreria TXS0108E
Parts:
- added U3: TXS0108EPWR-TSSOP20, Seeed-IC-2016:TSSOP20-0.65-6.5X4.4MM
Changed lines of the file:
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@@
 <layer number="112" name="tSilk" color="7" fill="1" visible="yes" active="yes"/>
 <layer number="113" name="IDFDebug" color="4" fill="1" visible="yes" active="yes"/>
+<layer number="114" name="FRNTMAAT1" color="7" fill="1" visible="yes" active="yes"/>
+<layer number="115" name="FRNTMAAT2" color="7" fill="1" visible="yes" active="yes"/>
 <layer number="116" name="Patch_BOT" color="9" fill="4" visible="yes" active="yes"/>
+<layer number="117" name="BACKMAAT1" color="7" fill="1" visible="yes" active="yes"/>
 <layer number="118" name="Rect_Pads" color="7" fill="1" visible="no" active="no"/>
+<layer number="119" name="KAP_TEKEN" color="7" fill="1" visible="yes" active="yes"/>
+<layer number="120" name="KAP_MAAT1" color="7" fill="1" visible="yes" active="yes"/>
 <layer number="121" name="_tsilk" color="7" fill="1" visible="yes" active="yes"/>
 <layer number="122" name="_bsilk" color="7" fill="1" visible="yes" active="yes"/>
@@
 <layer number="128" name="_bValues" color="7" fill="1" visible="yes" active="yes"/>
 <layer number="129" name="Mask" color="7" fill="1" visible="yes" active="yes"/>
+<layer number="130" name="SMDSTROOK" color="7" fill="1" visible="yes" active="yes"/>
 <layer number="131" name="tAdjust" color="7" fill="1" visible="yes" active="yes"/>
 <layer number="132" name="bAdjust" color="7" fill="1" visible="yes" active="yes"/>
+<layer number="133" name="bottom_silk" color="7" fill="1" visible="yes" active="yes"/>
 <layer number="144" name="Drill_legend" color="7" fill="1" visible="yes" active="yes"/>
 <layer number="150" name="Notes" color="7" fill="1" visible="yes" active="yes"/>
@@
 <element name="R7" library="rcl" package="R0805" value="0" x="-1.27" y="-200.66"/>
 <element name="U1" library="partes v2" package="LFCSP56" value="AD8192" x="-8.89" y="-196.85"/>
+<element name="U3" library="Seeed-IC-2016" package="TSSOP20-0.65-6.5X4.4MM" value="TXS0108EPWR-TSSOP20" x="-17.78" y="-199.39">
+<attribute name="MPN" value="TXS0108EPWR" x="-17.78" y="-199.39" size="1.778" layer="27" display="off"/>
+</element>
 </elements>
 <signals>

Commit message: avances pcb v2
Parts:
- removed Q4: MOSFET-NCHANNELBSS138, SparkFun-DiscreteSemi:SOT23-3
- removed U1: AD8192, partes v2:LFCSP56
- added C12, C13, C14: 100nF, rcl:C0805
- added C15: 470pF, rcl:C1206
- added C4: 100uF, rcl:C1206
- added MDL1: (no value), ESP8266-ESP12E:ESP8266-ESP12E
- added R10, R11, R12, R14, R8, R9: 10k, rcl:R0805
- R3, R6: value 10k -> 4.7k
- R4: value 4.7K -> 1k
Connections:
- net RELE1 renamed RELE
- removed net AMUXVCC: U1.47
- removed net AVCC: U1.1
- removed net AVCC1: U1.10
- removed net AVCC2: U1.33
- removed net AVCC3: U1.42
- removed net AVEE: U1.4
- removed net AVEE1: U1.13
- removed net AVEE2: U1.30
- removed net AVEE3: U1.39
- removed net AVEE4: U1.EXP
- removed net DVCC: U1.15
- removed net DVCC1: U1.21
- removed net DVEE: U1.52
- removed net RELE2: U2.25
- removed net RFID_INT: JP1.5
- removed net RFID_MISO: JP1.4
- removed net RFID_MOSI: JP1.3
- removed net RFID_PW: U2.9
- removed net RFID_RST: JP1.7
- removed net RFID_SCK: JP1.2
- removed net RFID_SS: JP1.1
- removed net RFID_TX: U2.32
- removed net VTTI: U1.7
- removed net VTTI1: U1.36
- removed net VTTO: U1.18
- removed net VTTO1: U1.24
- new net ESP_OC_NPROG: MDL1.12, R12.1
- new net ESP_OC_NRST: C15.1, MDL1.1, R9.1
- new net ESP_RX_3V3: MDL1.15, U3.6
- new net ESP_TX_3V3: MDL1.16, U3.7
- new net LVLSHF_OC_OE: R14.1, U3.10
- new net N$10: MDL1.3, R8.1
- new net N$13: MDL1.11, R11.1
- new net N$16: MDL1.10, R10.2
- new net N$8: U2.12, U3.20
- new net RFID_MISO_3V3: JP1.4, U3.5
- new net RFID_MOSI_3V3: JP1.3, U3.4
- new net RFID_OC_NRST: JP1.7, U2.11
- new net RFID_SCK_3V3: JP1.2, U3.3
- new net RFID_SS_3V3: JP1.1, U3.1
- net +3V3: now also C13.1, C14.1, C4.1, MDL1.8, R11.2, R12.2, R14.2, R8.2, R9.2, U3.2
- net +5V: now also C12.1, U3.19
- net GND: now also C12.2, C13.2, C14.2, C15.2, C4.2, MDL1.9, R10.1, U3.11
- net N$17: now also U3.18
- net N$18: now also U3.16
- net N$19: now also U3.17
- net N$21: now also U3.14
- net N$22: now also U3.15

Commit message: v2 esquematico semiterminado
Parts:
- added C16: 1000uF, rcl:E2,5-6
- added C17: 10uF, rcl:E2,5-6
- added D1: CD1206-S01575, diode:MINIMELF
- added J2, J3: HDMI, partes v2:HDMI
- added JP2: M025MM, SparkFun-Connectors:SCREWTERMINAL-5MM-2
- added K1: (no value), pimoroni-mechanical:RELAY-EE2
- added Q3: PMBT3904, diego:SOT-23-3
- added R15: 1k, rcl:R0805
- added R16: 10k, rcl:R0805
- added S1: (no value), SparkFun-Electromechanical:SWITCH-SPDT
- added U1: ADP3338AKCZ-3.3RL7, ADI-Phase-2:SOT230P700X180-4N
Connections:
- new net HDMI_IN_5V: J3.P$18, K1.4, R16.1
- new net N$15: D1.A, K1.12, Q3.2
- new net N$20: Q3.1, R15.2
- new net N$23: J2.P$3, J3.P$3
- new net N$24: J2.P$4, J3.P$4
- new net N$25: J2.P$6, J3.P$6
- new net N$26: J2.P$7, J3.P$7
- new net N$27: J2.P$9, J3.P$9
- new net N$28: J2.P$10, J3.P$10
- new net N$29: J2.P$12, J3.P$12
- new net N$30: J2.P$13, J3.P$13
- new net N$31: J2.P$15, J3.P$15
- new net N$32: J2.P$16, J3.P$16
- new net N$33: J2.P$19, J3.P$19
- new net N$34: R16.2, U2.25
- new net N$35: J2.P$18, K1.5
- new net N$36: JP2.1, S1.2
- new net N$9: J2.P$1, J3.P$1
- net +3V3: now also C17.+, U1.2, U1.4
- net +5V: now also C16.+, D1.C, K1.1, S1.1, U1.3
- net GND: now also C16.-, C17.-, J2.P$11, J2.P$17, J2.P$2, J2.P$20, J2.P$21, J2.P$22, J2.P$23, J2.P$5, J2.P$8, J3.P$11, J3.P$17, J3.P$2, J3.P$20, J3.P$21, J3.P$22, J3.P$23, J3.P$5, J3.P$8, JP2.2, Q3.3, U1.1
- net RELE: now also R15.1

Commit message: fram
Parts:
- added C18: 100nF, rcl:C0805
- added R17: 10k, rcl:R0805
- added U4: MB85RS16N, partes v2:SOP8
Connections:
- net HDMI_IN_5V renamed HDMI_A_5V
- removed net N$35: J2.P$18, K1.5
- new net HDMI_B_5V: J2.P$18, K1.5, R17.1
- new net N$37: R17.2, U2.26
- new net N$39: U3.8, U4.1
- new net N$40: U3.9, U4.7
- net +3V3: now also C18.1, U4.8
- net GND: now also C18.2, U4.4
- net RFID_MISO_3V3: now also U4.2
- net RFID_MOSI_3V3: now also U4.5
- net RFID_SCK_3V3: now also U4.6
Changed lines of the file:
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@@
 <?xml version="1.0" encoding="utf-8"?>
 <!DOCTYPE eagle SYSTEM "eagle.dtd">
-<eagle version="7.5.0">
+<eagle version="7.2.0">
 <drawing>
 <settings>
@@
 <element name="C16" library="rcl" package="E2,5-6" value="1000uF" x="-8.89" y="-384.81"/>
 <element name="C17" library="rcl" package="E2,5-6" value="10uF" x="-21.59" y="-393.7"/>
+<element name="R17" library="rcl" package="R0805" value="10k" x="-22.86" y="-400.05"/>
+<element name="U4" library="partes v2" package="SOP8" value="MB85RS16N" x="-30.48" y="-398.78"/>
+<element name="C18" library="rcl" package="C0805" value="100nF" x="-31.75" y="-406.4"/>
 </elements>
 <signals>
@@
 <contactref element="J2" pad="P$8"/>
 <contactref element="J2" pad="P$5"/>
+<contactref element="U4" pad="4"/>
+<contactref element="C18" pad="2"/>
 <wire x1="-18.1" y1="-226.06" x2="-18.1" y2="-232.41" width="0" layer="19" extent="1-1"/>
 <wire x1="-4.12" y1="-258.35" x2="-18.1" y2="-232.41" width="0" layer="19" extent="1-1"/>
@@
 <wire x1="-20.32" y1="-393.7" x2="-16.59" y2="-386.08" width="0" layer="19" extent="1-1"/>
 <wire x1="-7.62" y1="-384.81" x2="-16.59" y2="-386.08" width="0" layer="19" extent="1-1"/>
+<wire x1="-28.575" y1="-401.38" x2="-20.32" y2="-393.7" width="0" layer="19" extent="1-1"/>
+<wire x1="-30.8" y1="-406.4" x2="-28.575" y2="-401.38" width="0" layer="19" extent="1-1"/>
 <wire x1="1.59" y1="-96.52" x2="8.89" y2="-132.08" width="0" layer="19" extent="1-1"/>
 <wire x1="3.49" y1="-68.58" x2="1.59" y2="-96.52" width="0" layer="19" extent="1-1"/>
@@
 <contactref element="JP1" pad="4"/>
 <contactref element="U3" pad="5"/>
+<contactref element="U4" pad="2"/>
 <wire x1="6.35" y1="-195.58" x2="-18.105" y2="-202.455" width="0" layer="19" extent="1-1"/>
+<wire x1="-31.115" y1="-401.38" x2="-18.105" y2="-202.455" width="0" layer="19" extent="1-1"/>
 </signal>
 <signal name="RFID_MOSI_3V3">
 <contactref element="JP1" pad="3"/>
 <contactref element="U3" pad="4"/>
+<contactref element="U4" pad="5"/>
 <wire x1="3.81" y1="-195.58" x2="-18.755" y2="-202.455" width="0" layer="19" extent="1-1"/>
+<wire x1="-28.575" y1="-396.18" x2="-18.755" y2="-202.455" width="0" layer="19" extent="1-1"/>
 </signal>
 <signal name="RFID_SCK_3V3">
 <contactref element="JP1" pad="2"/>
 <contactref element="U3" pad="3"/>
+<contactref element="U4" pad="6"/>
 <wire x1="1.27" y1="-195.58" x2="-19.405" y2="-202.455" width="0" layer="19" extent="1-1"/>
+<wire x1="-29.845" y1="-396.18" x2="-19.405" y2="-202.455" width="0" layer="19" extent="1-1"/>
 </signal>
 <signal name="RFID_SS_3V3">
@@
 <contactref element="U1" pad="2"/>
 <contactref element="C17" pad="+"/>
+<contactref element="C18" pad="1"/>
+<contactref element="U4" pad="8"/>
 <wire x1="-20.32" y1="-258.35" x2="-20" y2="-232.41" width="0" layer="19" extent="1-1"/>
 <wire x1="-20.45" y1="-265.43" x2="-20.32" y2="-258.35" width="0" layer="19" extent="1-1"/>
@@
 <wire x1="-22.2504" y1="-374.65" x2="-15.8496" y2="-374.65" width="0" layer="19" extent="1-1"/>
 <wire x1="-22.86" y1="-393.7" x2="-22.2504" y2="-374.65" width="0" layer="19" extent="1-1"/>
+<wire x1="-32.385" y1="-396.18" x2="-22.86" y2="-393.7" width="0" layer="19" extent="1-1"/>
+<wire x1="-32.7" y1="-406.4" x2="-32.385" y2="-396.18" width="0" layer="19" extent="1-1"/>
 </signal>
 <signal name="N$7">
@@
 <wire x1="-18.47" y1="-316.29" x2="-18.47" y2="-332.8" width="0" layer="19" extent="1-1"/>
 </signal>
-<signal name="HDMI_IN_5V">
+<signal name="HDMI_A_5V">
 <contactref element="J3" pad="P$18"/>
 <contactref element="K1" pad="4"/>
@@
 <wire x1="-12.8" y1="-297.015" x2="-17.97" y2="-332.8" width="0" layer="19" extent="1-1"/>
 </signal>
-<signal name="N$35">
+<signal name="HDMI_B_5V">
 <contactref element="K1" pad="5"/>
 <contactref element="J2" pad="P$18"/>
+<contactref element="R17" pad="1"/>
+<wire x1="-17.97" y1="-316.29" x2="-23.81" y2="-400.05" width="0" layer="19" extent="1-1"/>
 <wire x1="-10.26" y1="-297.015" x2="-17.97" y2="-316.29" width="0" layer="19" extent="1-1"/>
 </signal>
@@
 <wire x1="-20.32" y1="-361.95" x2="-21.59" y2="-386.08" width="0" layer="19" extent="1-1"/>
 </signal>
+<signal name="N$37">
+<contactref element="U2" pad="26"/>
+<contactref element="R17" pad="2"/>
+<wire x1="7.08" y1="-2.0574" x2="-21.91" y2="-400.05" width="0" layer="19" extent="1-1"/>
+</signal>
+<signal name="N$39">
+<contactref element="U4" pad="1"/>
+<contactref element="U3" pad="8"/>
+<wire x1="-32.385" y1="-401.38" x2="-16.155" y2="-202.455" width="0" layer="19" extent="1-1"/>
+</signal>
+<signal name="N$40">
+<contactref element="U4" pad="7"/>
+<contactref element="U3" pad="9"/>
+<wire x1="-31.115" y1="-396.18" x2="-15.505" y2="-202.455" width="0" layer="19" extent="1-1"/>
+</signal>
 </signals>
