File: Hardware/pcb v2/sch y brd/pcb v2.brd (EAGLE design)
At the start: 160 x 100 mm, 56 parts, among them J1 AVR_SPI_PRG_6PTH, J2 HDMI, J3 HDMI, Q1 32.768kHz 12.5pF, Q2 PMBT3904, Q3 PMBT3904, U1 ADP3338AKCZ-3.3RL7, U2 ATMEGA328P, U3 TXS0108EPWR-TSSOP20, U4 MB85RS16N, Y1 16Mhz

Commit message: v2 esquematico completo
Parts:
- added C19: 1uF, rcl:C0805
- added C20: 100nF, rcl:C0805
- added J4: HDMI, partes v2:HDMI
- added JP3: (no value), SparkFun-Connectors:1X08
- added JP4: 2X6 FEMALE, SparkFun-Connectors:2X6
- C10: value 100nF -> 10uF; device rcl:C0805 -> rcl:C1206
- C11: device rcl:C0805 -> rcl:C1206
- C15: value 470pF -> 10uF; device rcl:C1206 -> rcl:E2,5-6
- C17: value 10uF -> 100nF; device rcl:E2,5-6 -> rcl:C0805
- C18: value 100nF -> 10uF; device rcl:C0805 -> rcl:E2,5-6
- C4: value 100uF -> 100nF; device rcl:C1206 -> rcl:C0805
- C5, C6: value 100nF -> 22pF; device rcl:C0805 -> rcl:C1206
- C7: value 22pF -> 100nF; device rcl:C1206 -> rcl:C0805
- C8: value 22pF -> 470pF
- C9: value 100nF -> 100uF; device rcl:C0805 -> rcl:C1206
- J2: value HDMI -> 1981584-1; device partes v2:HDMI -> con-usb:1981584-1
- JP1: device SparkFun-Connectors:1X08 -> SparkFun-Connectors:JST-3-SMD
- JP2: value M025MM -> FEMALE 2x3; device SparkFun-Connectors:SCREWTERMINAL-5MM-2 -> SparkFun-Connectors:2X3
- Q1: value 32.768kHz 12.5pF -> PMBT3904; device crystal:TC26H -> diego:SOT-23-3
- Q3: value PMBT3904 -> 32.768kHz 12.5pF; device diego:SOT-23-3 -> crystal:TC26H
- R1: value 1K -> NO(10k)
- R10: value 10k -> 0
- R12, R9: value 10k -> 1k
- R13: value 10K -> 1K
- R15, R4: value 1k -> 10k
- R16, R17: value 10k -> 4.7k
- R3, R6: value 4.7k -> 10k
- R5: value 1K -> 10k
- R7: value 0 -> 10k
- S1: value (none) -> SWITCH-MOMENTARY-2SMD; device SparkFun-Electromechanical:SWITCH-SPDT -> SparkFun-Electromechanical:TACTILE-SWITCH-SMD
- U1: value ADP3338AKCZ-3.3RL7 -> ATMEGA328P; device ADI-Phase-2:SOT230P700X180-4N -> SparkFun-DigitalIC:TQFP32-08
- U2: value ATMEGA328P -> TXS0108EPWR-TSSOP20; device SparkFun-DigitalIC:TQFP32-08 -> Seeed-IC-2016:TSSOP20-0.65-6.5X4.4MM
- U3: value TXS0108EPWR-TSSOP20 -> MB85RS16N; device Seeed-IC-2016:TSSOP20-0.65-6.5X4.4MM -> partes v2:SOP8
- U4: value MB85RS16N -> ADP3338AKCZ-3.3RL7; device partes v2:SOP8 -> ADI-Phase-2:SOT230P700X180-4N
- moved R1 376.2 mm to (-31.8, -471.2)
- moved U1 369.1 mm to (5.08, -6.35)
- moved JP1 319.1 mm to (-38.4, -512.5)
- moved C10 316.2 mm to (-31.8, -458.5)
- moved C11 278.5 mm to (-31.8, -464.8)
- moved R17 260.5 mm to (29.2, -144.8)
- moved D1 260.3 mm to (2.54, -49.5)
- moved D2 260.3 mm to (-22.9, -308.6)
- moved C8 243.9 mm to (-19.1, -278.1)
- moved C4 229.6 mm to (2.54, -36.8)
- moved R10 214.0 mm to (-22.9, -478.8), turned to 180 degrees
- moved R16 207.5 mm to (19.1, -144.8)
- moved U3 199.8 mm to (-30.5, -398.8)
- moved U2 194.4 mm to (-17.8, -199.4)
- moved Q1 175.0 mm to (-24.1, -295.9)
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- renumbered U$1 to U5
Connections:
- removed net N$36: JP2.1, S1.2
- removed net N$40: U3.9, U4.7
- removed net RST_ATM_FLANCO: C9.1, R1.2
- new net ADC6: JP4.3, U1.19
- new net ADC7: JP4.5, U1.22
- new net BOTON: R15.1, S1.1, U1.32
- new net N$41: U1.10, U2.13
- new net PB2: JP4.6, U1.14
- new net PD3: JP4.7, U1.1
- new net PD4: JP4.9, U1.2
- new net PD5: JP4.4, U1.9
- new net RST_ATM_3V3: MDL1.13, U2.9
- net +3V3: now also C10.1, C11.1, C12.1, C17.1, C18.+, C9.1, JP3.8, JP4.2, R2.2, R4.2, R5.2, R6.2, U2.2, U3.3, U3.7, U3.8, U4.2, U4.4; no longer C13.1, C17.+, C18.1, C4.1, JP1.8, R12.2, R14.2, R8.2, R9.2, U1.2, U1.4, U3.2, U4.8
- net +5V: now also C1.1, C13.1, C15.+, C19.1, C20.1, J2.1, JP1.3, JP4.1, R1.2, R13.2, R14.2, R15.2, R16.2, R17.2, U1.18, U1.4, U1.6, U2.19, U4.3; no longer C10.1, C11.1, C12.1, C5.1, R13.1, R2.2, R3.2, R5.2, R6.2, S1.1, U1.3, U2.18, U2.4, U2.6, U3.19
- net BUZZER: now also R12.1, U1.23; no longer R4.1, U2.23
- net ESP_OC_NPROG: now also JP2.5, R2.1; no longer R12.1
- net ESP_OC_NRST: now also C8.1, JP2.4, R6.1; no longer C15.1, R9.1
- net ESP_RX_3V3: now also JP2.1, U2.6; no longer U3.6
- net ESP_TX_3V3: now also JP2.2, U2.7; no longer U3.7
- net GND: now also C15.-, C17.2, C18.-, C19.2, C20.2, C9.2, J2.5, J2.S1, J2.S2, J2.S3, J2.S4, J4.P$11, J4.P$17, J4.P$2, J4.P$20, J4.P$21, J4.P$22, J4.P$23, J4.P$5, J4.P$8, JP1.1, JP3.6, JP4.11, JP4.12, Q1.3, R3.1, S1.3, U1.21, U1.3, U1.5, U2.11, U3.4, U4.1; no longer C15.2, C17.-, C18.2, J2.P$11, J2.P$17, J2.P$2, J2.P$20, J2.P$21, J2.P$22, J2.P$23, J2.P$5, J2.P$8, JP1.6, JP2.2, Q3.3, R1.1, R10.1, U1.1, U2.21, U2.3, U2.5, U3.11, U4.4
- net HDMI_A_5V: now also R7.1; no longer R16.1
- net HDMI_B_5V: now also J4.P$18, R8.1; no longer J2.P$18, R17.1
- net LED: now also JP1.2, U1.13; no longer U2.13
- net LVLSHF_OC_OE: now also JP2.3, R11.1, U2.10; no longer R14.1, U3.10
- net N$1: now also R12.2; no longer R4.2
- net N$10: now also R5.1; no longer R8.1
- net N$11: now also C5.1, U1.7; no longer C7.1, U2.7
- net N$12: now also C6.1, U1.8; no longer C8.1, U2.8
- net N$13: now also R4.1; no longer R11.1
- net N$14: now also C4.1, U1.20; no longer C6.1, U2.20
- net N$15: now also D2.A, Q1.2; no longer D1.A, Q3.2
- net N$16: now also R3.2; no longer R10.2
- net N$17: now also U1.17, U2.18; no longer U2.17, U3.18
- net N$18: now also U1.16; no longer U3.16
- net N$19: now also U1.15, U2.17; no longer U2.15, U3.17
- net N$2: now also Q3.2; no longer Q1.2
- net N$20: now also Q1.1, R9.2; no longer Q3.1, R15.2
- net N$21: now also U1.30, U2.14; no longer U2.30, U3.14
- net N$22: now also U1.31, U2.15; no longer U2.31, U3.15
- net N$23: now also J4.P$3; no longer J2.P$3
- net N$24: now also J4.P$4; no longer J2.P$4
- net N$25: now also J4.P$6; no longer J2.P$6
- net N$26: now also J4.P$7; no longer J2.P$7
- net N$27: now also J4.P$9; no longer J2.P$9
- net N$28: now also J4.P$10; no longer J2.P$10
- net N$29: now also J4.P$12; no longer J2.P$12
- net N$3: now also Q3.1; no longer Q1.1
- net N$30: now also J4.P$13; no longer J2.P$13
- net N$31: now also J4.P$15; no longer J2.P$15
- net N$32: now also J4.P$16; no longer J2.P$16
- net N$33: now also J4.P$19; no longer J2.P$19
- net N$34: now also R7.2, U1.25; no longer R16.2, U2.25
- net N$37: now also R8.2, U1.26; no longer R17.2, U2.26
- net N$39: now also U2.8, U3.1; no longer U3.8, U4.1
- net N$5: now also R13.1; no longer R5.1
- net N$6: now also R14.1; no longer R2.1
- net N$7: now also R10.1, U2.12; no longer C9.2, R7.2
- net N$8: now also U1.12, U2.20; no longer U2.12, U3.20
- net N$9: now also J4.P$1; no longer J2.P$1
- net RELE: now also R9.1, U1.24; no longer R15.1, U2.24
- net RFID_MISO_3V3: now also JP3.4, U2.5, U3.2; no longer JP1.4, U3.5, U4.2
- net RFID_MOSI_3V3: now also JP3.3, U2.4, U3.5; no longer JP1.3, U3.4, U4.5
- net RFID_OC_NRST: now also JP3.7, U1.11; no longer JP1.7, U2.11
- net RFID_SCK_3V3: now also JP3.2, U2.3, U3.6; no longer JP1.2, U3.3, U4.6
- net RFID_SS_3V3: now also JP3.1, U2.1; no longer JP1.1, U3.1
- net RST_ATM: now also C7.1, D1.A, R1.1, R10.2, U1.29; no longer C1.1, D2.A, R13.2, R7.1, U2.29
- net SCL: now also JP4.10, R16.1, U1.28; no longer R3.1, U2.28
- net SDA: now also JP4.8, R17.1, U1.27; no longer R6.1, U2.27
