File: Hardware/pcb v2/sch y brd/pcb v2.sch (EAGLE design)
At the start: 23 parts, among them J1 AVR_SPI_PRG_6PTH, Q1 32.768kHz 12.5pF, Q4 MOSFET-NCHANNELBSS138, U2 ATMEGA328P, Y1 16Mhz

Commit message: pcb v2 buzzer
Parts:
- added C11: 1uF, rcl:C-USC0805
- added Q2: PMBT3904, diego:PMBT3904
- added R4: 4.7K, rcl:R-US_R0805
- added R5: 1K, rcl:R-US_R0805
- added SG1: BUZZERPTH, SparkFun-Electromechanical:BUZZERPTH
Connections:
- net LED_R renamed LED
- removed net LED_B: U2.PD6(AIN0)
- removed net LED_G: U2.PB2(SS/OC1B)
- new net N$1: Q2.B, R4.2
- new net N$5: Q2.C, R5.1, SG1.2
- net +5V: now also C11.1, R5.2, SG1.1
- net BUZZER: now also R4.1
- net GND: now also C11.2, Q2.E
Changed lines of the file:
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@@
 <setting verticaltext="up"/>
 </settings>
-<grid distance="0.1" unitdist="inch" unit="inch" style="dots" multiple="1" display="yes" altdistance="0.01" altunitdist="inch" altunit="inch"/>
+<grid distance="0.1" unitdist="inch" unit="inch" style="lines" multiple="1" display="no" altdistance="0.01" altunitdist="inch" altunit="inch"/>
 <layers>
 <layer number="1" name="Top" color="4" fill="1" visible="no" active="no"/>
@@
 <part name="C10" library="rcl" deviceset="C-US" device="C0805" value="100nF"/>
 <part name="GND10" library="supply1" deviceset="GND" device=""/>
+<part name="SG1" library="SparkFun-Electromechanical" deviceset="BUZZER" device="PTH"/>
+<part name="GND7" library="supply1" deviceset="GND" device=""/>
+<part name="Q2" library="diego" deviceset="PMBT3904" device=""/>
+<part name="R4" library="rcl" deviceset="R-US_" device="R0805" value="4.7K"/>
+<part name="R5" library="rcl" deviceset="R-US_" device="R0805" value="1K"/>
+<part name="P+1" library="supply1" deviceset="+5V" device=""/>
+<part name="C11" library="rcl" deviceset="C-US" device="C0805" value="1uF"/>
+<part name="GND4" library="supply1" deviceset="GND" device=""/>
 </parts>
 <sheets>
@@
 <instance part="C10" gate="G$1" x="86.36" y="193.04"/>
 <instance part="GND10" gate="1" x="86.36" y="180.34"/>
+<instance part="SG1" gate="G$1" x="205.74" y="190.5" smashed="yes" rot="R270">
+<attribute name="NAME" x="210.82" y="193.04" size="1.778" layer="95" rot="R270"/>
+<attribute name="VALUE" x="207.01" y="195.58" size="1.778" layer="96"/>
+</instance>
+<instance part="GND7" gate="1" x="195.58" y="160.02"/>
+<instance part="Q2" gate="G$1" x="193.04" y="172.72"/>
+<instance part="R4" gate="G$1" x="180.34" y="172.72"/>
+<instance part="R5" gate="G$1" x="195.58" y="187.96" rot="R90"/>
+<instance part="P+1" gate="1" x="195.58" y="200.66"/>
+<instance part="C11" gate="G$1" x="180.34" y="190.5"/>
+<instance part="GND4" gate="1" x="180.34" y="180.34"/>
 </instances>
 <busses>
@@
 <pinref part="C10" gate="G$1" pin="2"/>
 <wire x1="86.36" y1="187.96" x2="86.36" y2="182.88" width="0.1524" layer="91"/>
+</segment>
+<segment>
+<pinref part="GND7" gate="1" pin="GND"/>
+<pinref part="Q2" gate="G$1" pin="E"/>
+<wire x1="195.58" y1="162.56" x2="195.58" y2="167.64" width="0.1524" layer="91"/>
+</segment>
+<segment>
+<pinref part="C11" gate="G$1" pin="2"/>
+<wire x1="180.34" y1="185.42" x2="180.34" y2="182.88" width="0.1524" layer="91"/>
+<pinref part="GND4" gate="1" pin="GND"/>
 </segment>
 </net>
@@
 <wire x1="109.22" y1="198.12" x2="109.22" y2="193.04" width="0.1524" layer="91"/>
 </segment>
+<segment>
+<pinref part="R5" gate="G$1" pin="2"/>
+<pinref part="P+1" gate="1" pin="+5V"/>
+<wire x1="195.58" y1="193.04" x2="195.58" y2="195.58" width="0.1524" layer="91"/>
+<pinref part="SG1" gate="G$1" pin="1"/>
+<wire x1="195.58" y1="195.58" x2="195.58" y2="198.12" width="0.1524" layer="91"/>
+<wire x1="203.2" y1="190.5" x2="200.66" y2="190.5" width="0.1524" layer="91"/>
+<wire x1="200.66" y1="190.5" x2="200.66" y2="195.58" width="0.1524" layer="91"/>
+<wire x1="200.66" y1="195.58" x2="195.58" y2="195.58" width="0.1524" layer="91"/>
+<junction x="195.58" y="195.58"/>
+<pinref part="C11" gate="G$1" pin="1"/>
+<wire x1="180.34" y1="193.04" x2="180.34" y2="195.58" width="0.1524" layer="91"/>
+<wire x1="180.34" y1="195.58" x2="195.58" y2="195.58" width="0.1524" layer="91"/>
+</segment>
 </net>
 <net name="RFID_PW" class="0">
@@
 <wire x1="121.92" y1="96.52" x2="127" y2="96.52" width="0.1524" layer="91"/>
 <label x="127" y="96.52" size="1.778" layer="95" xref="yes"/>
+</segment>
+<segment>
+<pinref part="R4" gate="G$1" pin="1"/>
+<wire x1="175.26" y1="172.72" x2="170.18" y2="172.72" width="0.1524" layer="91"/>
+<label x="170.18" y="172.72" size="1.778" layer="95" rot="R180" xref="yes"/>
 </segment>
 </net>
@@
 </segment>
 </net>
-<net name="LED_R" class="0">
+<net name="LED" class="0">
 <segment>
 <pinref part="U2" gate="G$1" pin="PB1(OC1A)"/>
-<wire x1="116.84" y1="43.18" x2="124.46" y2="43.18" width="0.1524" layer="91"/>
-<wire x1="124.46" y1="43.18" x2="124.46" y2="45.72" width="0.1524" layer="91"/>
-<wire x1="124.46" y1="45.72" x2="127" y2="45.72" width="0.1524" layer="91"/>
-<label x="127" y="45.72" size="1.778" layer="95" xref="yes"/>
-</segment>
-</net>
-<net name="LED_G" class="0">
-<segment>
-<pinref part="U2" gate="G$1" pin="PB2(SS/OC1B)"/>
-<wire x1="116.84" y1="40.64" x2="127" y2="40.64" width="0.1524" layer="91"/>
-<label x="127" y="40.64" size="1.778" layer="95" xref="yes"/>
-</segment>
-</net>
-<net name="LED_B" class="0">
-<segment>
-<pinref part="U2" gate="G$1" pin="PD6(AIN0)"/>
-<wire x1="116.84" y1="53.34" x2="121.92" y2="53.34" width="0.1524" layer="91"/>
-<wire x1="121.92" y1="53.34" x2="121.92" y2="50.8" width="0.1524" layer="91"/>
-<wire x1="121.92" y1="50.8" x2="127" y2="50.8" width="0.1524" layer="91"/>
-<label x="127" y="50.8" size="1.778" layer="95" xref="yes"/>
+<wire x1="116.84" y1="43.18" x2="127" y2="43.18" width="0.1524" layer="91"/>
+<label x="127" y="43.18" size="1.778" layer="95" xref="yes"/>
 </segment>
 </net>
@@
 </segment>
 </net>
+<net name="N$1" class="0">
+<segment>
+<pinref part="R4" gate="G$1" pin="2"/>
+<pinref part="Q2" gate="G$1" pin="B"/>
+<wire x1="185.42" y1="172.72" x2="190.5" y2="172.72" width="0.1524" layer="91"/>
+</segment>
+</net>
+<net name="N$5" class="0">
+<segment>
+<pinref part="Q2" gate="G$1" pin="C"/>
+<pinref part="R5" gate="G$1" pin="1"/>
+<wire x1="195.58" y1="177.8" x2="195.58" y2="180.34" width="0.1524" layer="91"/>
+<pinref part="SG1" gate="G$1" pin="2"/>
+<wire x1="195.58" y1="180.34" x2="195.58" y2="182.88" width="0.1524" layer="91"/>
+<wire x1="203.2" y1="187.96" x2="200.66" y2="187.96" width="0.1524" layer="91"/>
+<wire x1="200.66" y1="187.96" x2="200.66" y2="180.34" width="0.1524" layer="91"/>
+<wire x1="200.66" y1="180.34" x2="195.58" y2="180.34" width="0.1524" layer="91"/>
+<junction x="195.58" y="180.34"/>
+</segment>
+</net>

Commit message: pcb v2 rfid
Parts:
- added JP1: (no value), SparkFun-Connectors:M081X08
Connections:
- new net +3V3: JP1.8
- new net RFID_INT: JP1.5
- new net RFID_MISO: JP1.4
- new net RFID_MOSI: JP1.3
- new net RFID_RST: JP1.7
- new net RFID_SCK: JP1.2
- new net RFID_SS: JP1.1
- net GND: now also JP1.6
Changed lines of the file:
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@@
 <setting verticaltext="up"/>
 </settings>
-<grid distance="0.1" unitdist="inch" unit="inch" style="lines" multiple="1" display="no" altdistance="0.01" altunitdist="inch" altunit="inch"/>
+<grid distance="0.1" unitdist="inch" unit="inch" style="dots" multiple="1" display="yes" altdistance="0.01" altunitdist="inch" altunit="inch"/>
 <layers>
 <layer number="1" name="Top" color="4" fill="1" visible="no" active="no"/>
@@
 <part name="C11" library="rcl" deviceset="C-US" device="C0805" value="1uF"/>
 <part name="GND4" library="supply1" deviceset="GND" device=""/>
+<part name="JP1" library="SparkFun-Connectors" deviceset="M08" device="1X08"/>
+<part name="GND5" library="supply1" deviceset="GND" device=""/>
+<part name="+3V2" library="supply1" deviceset="+3V3" device=""/>
 </parts>
 <sheets>
@@
 <instance part="C11" gate="G$1" x="180.34" y="190.5"/>
 <instance part="GND4" gate="1" x="180.34" y="180.34"/>
+<instance part="JP1" gate="G$1" x="193.04" y="134.62" rot="R180"/>
+<instance part="GND5" gate="1" x="172.72" y="116.84"/>
+<instance part="+3V2" gate="G$1" x="170.18" y="137.16"/>
 </instances>
 <busses>
@@
 <wire x1="180.34" y1="185.42" x2="180.34" y2="182.88" width="0.1524" layer="91"/>
 <pinref part="GND4" gate="1" pin="GND"/>
+</segment>
+<segment>
+<pinref part="JP1" gate="G$1" pin="6"/>
+<wire x1="187.96" y1="129.54" x2="172.72" y2="129.54" width="0.1524" layer="91"/>
+<wire x1="172.72" y1="129.54" x2="172.72" y2="119.38" width="0.1524" layer="91"/>
+<pinref part="GND5" gate="1" pin="GND"/>
 </segment>
 </net>
@@
 </segment>
 </net>
+<net name="RFID_MISO" class="0">
+<segment>
+<pinref part="JP1" gate="G$1" pin="4"/>
+<wire x1="187.96" y1="134.62" x2="185.42" y2="134.62" width="0.1524" layer="91"/>
+<label x="185.42" y="134.62" size="1.016" layer="95" rot="R180" xref="yes"/>
+</segment>
+</net>
+<net name="RFID_MOSI" class="0">
+<segment>
+<pinref part="JP1" gate="G$1" pin="3"/>
+<wire x1="187.96" y1="137.16" x2="185.42" y2="137.16" width="0.1524" layer="91"/>
+<label x="185.42" y="137.16" size="1.016" layer="95" rot="R180" xref="yes"/>
+</segment>
+</net>
+<net name="RFID_SCK" class="0">
+<segment>
+<pinref part="JP1" gate="G$1" pin="2"/>
+<wire x1="187.96" y1="139.7" x2="185.42" y2="139.7" width="0.1524" layer="91"/>
+<label x="185.42" y="139.7" size="1.016" layer="95" rot="R180" xref="yes"/>
+</segment>
+</net>
+<net name="RFID_SS" class="0">
+<segment>
+<pinref part="JP1" gate="G$1" pin="1"/>
+<wire x1="187.96" y1="142.24" x2="185.42" y2="142.24" width="0.1524" layer="91"/>
+<label x="185.42" y="142.24" size="1.016" layer="95" rot="R180" xref="yes"/>
+</segment>
+</net>
+<net name="RFID_INT" class="0">
+<segment>
+<pinref part="JP1" gate="G$1" pin="5"/>
+<wire x1="187.96" y1="132.08" x2="185.42" y2="132.08" width="0.1524" layer="91"/>
+<label x="185.42" y="132.08" size="1.016" layer="95" rot="R180" xref="yes"/>
+</segment>
+</net>
+<net name="RFID_RST" class="0">
+<segment>
+<pinref part="JP1" gate="G$1" pin="7"/>
+<wire x1="187.96" y1="127" x2="185.42" y2="127" width="0.1524" layer="91"/>
+<label x="185.42" y="127" size="1.016" layer="95" rot="R180" xref="yes"/>
+</segment>
+</net>
+<net name="+3V3" class="0">
+<segment>
+<pinref part="JP1" gate="G$1" pin="8"/>
+<wire x1="187.96" y1="124.46" x2="170.18" y2="124.46" width="0.1524" layer="91"/>
+<wire x1="170.18" y1="124.46" x2="170.18" y2="134.62" width="0.1524" layer="91"/>
+<pinref part="+3V2" gate="G$1" pin="+3V3"/>
+</segment>
+</net>

Commit message: libreria AD8192
Parts:
- removed RESET-EN1: (no value), jumper:SJ
- added R7: 0, rcl:R-US_R0805
- added U1: AD8192, partes v2:AD8192
Connections:
- new net N$7: C9.2, R7.2
- net RST_ATM: now also R7.1; no longer C9.2, RESET-EN1.1, RESET-EN1.2
Changed lines of the file:
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@@
 <part name="C2" library="rcl" deviceset="C-US" device="C0805" value="100nF"/>
 <part name="C3" library="rcl" deviceset="C-US" device="C0805" value="100nF"/>
-<part name="RESET-EN1" library="jumper" deviceset="SJ" device=""/>
 <part name="R1" library="rcl" deviceset="R-US_" device="R0805" value="1K"/>
 <part name="GND2" library="supply1" deviceset="GND" device=""/>
@@
 <part name="GND5" library="supply1" deviceset="GND" device=""/>
 <part name="+3V2" library="supply1" deviceset="+3V3" device=""/>
+<part name="R7" library="rcl" deviceset="R-US_" device="R0805" value="0"/>
+<part name="U1" library="partes v2" deviceset="AD8192" device=""/>
 </parts>
 <sheets>
@@
 <instance part="C2" gate="G$1" x="27.94" y="71.12"/>
 <instance part="C3" gate="G$1" x="17.78" y="71.12"/>
-<instance part="RESET-EN1" gate="1" x="43.18" y="129.54"/>
 <instance part="R1" gate="G$1" x="17.78" y="119.38" rot="R90"/>
 <instance part="GND2" gate="1" x="17.78" y="106.68"/>
@@
 <instance part="GND5" gate="1" x="172.72" y="116.84"/>
 <instance part="+3V2" gate="G$1" x="170.18" y="137.16"/>
+<instance part="R7" gate="G$1" x="43.18" y="129.54" rot="R180"/>
+<instance part="U1" gate="G$1" x="238.76" y="71.12"/>
 </instances>
 <busses>
@@
 <wire x1="73.66" y1="116.84" x2="73.66" y2="114.3" width="0.1524" layer="91"/>
 <junction x="63.5" y="116.84"/>
-<pinref part="RESET-EN1" gate="1" pin="2"/>
-<wire x1="48.26" y1="129.54" x2="50.8" y2="129.54" width="0.1524" layer="91"/>
 <junction x="63.5" y="129.54"/>
-<pinref part="RESET-EN1" gate="1" pin="1"/>
-<wire x1="50.8" y1="129.54" x2="63.5" y2="129.54" width="0.1524" layer="91"/>
-<wire x1="30.48" y1="129.54" x2="35.56" y2="129.54" width="0.1524" layer="91"/>
-<wire x1="35.56" y1="129.54" x2="38.1" y2="129.54" width="0.1524" layer="91"/>
-<wire x1="35.56" y1="129.54" x2="35.56" y2="124.46" width="0.1524" layer="91"/>
-<wire x1="35.56" y1="124.46" x2="50.8" y2="124.46" width="0.1524" layer="91"/>
-<junction x="35.56" y="129.54"/>
-<wire x1="50.8" y1="124.46" x2="50.8" y2="129.54" width="0.1524" layer="91"/>
-<junction x="50.8" y="129.54"/>
-<pinref part="C9" gate="G$1" pin="2"/>
+<wire x1="48.26" y1="129.54" x2="63.5" y2="129.54" width="0.1524" layer="91"/>
+<pinref part="R7" gate="G$1" pin="1"/>
 </segment>
 </net>
@@
 </segment>
 </net>
+<net name="N$7" class="0">
+<segment>
+<wire x1="30.48" y1="129.54" x2="38.1" y2="129.54" width="0.1524" layer="91"/>
+<pinref part="C9" gate="G$1" pin="2"/>
+<pinref part="R7" gate="G$1" pin="2"/>
+</segment>
+</net>

Commit message: libreria TXS0108E
Parts:
- added U3: TXS0108EPWR-TSSOP20, Seeed-IC-2016:LOGIC-TXS0108EPWR(TSSOP20)
Changed lines of the file:
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@@
 <setting verticaltext="up"/>
 </settings>
-<grid distance="0.1" unitdist="inch" unit="inch" style="dots" multiple="1" display="yes" altdistance="0.01" altunitdist="inch" altunit="inch"/>
+<grid distance="0.1" unitdist="inch" unit="inch" style="lines" multiple="1" display="no" altdistance="0.01" altunitdist="inch" altunit="inch"/>
 <layers>
 <layer number="1" name="Top" color="4" fill="1" visible="no" active="no"/>
@@
 <layer number="112" name="tSilk" color="7" fill="1" visible="yes" active="yes"/>
 <layer number="113" name="IDFDebug" color="4" fill="1" visible="yes" active="yes"/>
+<layer number="114" name="FRNTMAAT1" color="7" fill="1" visible="yes" active="yes"/>
+<layer number="115" name="FRNTMAAT2" color="7" fill="1" visible="yes" active="yes"/>
 <layer number="116" name="Patch_BOT" color="9" fill="4" visible="yes" active="yes"/>
+<layer number="117" name="BACKMAAT1" color="7" fill="1" visible="yes" active="yes"/>
 <layer number="118" name="Rect_Pads" color="7" fill="1" visible="no" active="no"/>
+<layer number="119" name="KAP_TEKEN" color="7" fill="1" visible="yes" active="yes"/>
+<layer number="120" name="KAP_MAAT1" color="7" fill="1" visible="yes" active="yes"/>
 <layer number="121" name="_tsilk" color="7" fill="1" visible="yes" active="yes"/>
 <layer number="122" name="_bsilk" color="7" fill="1" visible="yes" active="yes"/>
@@
 <layer number="128" name="_bValues" color="7" fill="1" visible="yes" active="yes"/>
 <layer number="129" name="Mask" color="7" fill="1" visible="yes" active="yes"/>
+<layer number="130" name="SMDSTROOK" color="7" fill="1" visible="yes" active="yes"/>
 <layer number="131" name="tAdjust" color="7" fill="1" visible="yes" active="yes"/>
 <layer number="132" name="bAdjust" color="7" fill="1" visible="yes" active="yes"/>
+<layer number="133" name="bottom_silk" color="7" fill="1" visible="yes" active="yes"/>
 <layer number="144" name="Drill_legend" color="7" fill="1" visible="yes" active="yes"/>
 <layer number="150" name="Notes" color="7" fill="1" visible="yes" active="yes"/>
@@
 <part name="R7" library="rcl" deviceset="R-US_" device="R0805" value="0"/>
 <part name="U1" library="partes v2" deviceset="AD8192" device=""/>
+<part name="U3" library="Seeed-IC-2016" deviceset="LOGIC-TXS0108EPWR(TSSOP20)" device="" value="TXS0108EPWR-TSSOP20"/>
 </parts>
 <sheets>
@@
 <instance part="R7" gate="G$1" x="43.18" y="129.54" rot="R180"/>
 <instance part="U1" gate="G$1" x="238.76" y="71.12"/>
+<instance part="U3" gate="G$1" x="144.78" y="127"/>
 </instances>
 <busses>

Commit message: avances pcb v2
Parts:
- removed Q4: MOSFET-NCHANNELBSS138, SparkFun-DiscreteSemi:MOSFET-NCHANNELBSS138
- removed U1: AD8192, partes v2:AD8192
- added C12, C13, C14: 100nF, rcl:C-USC0805
- added C15: 470pF, rcl:C-USC1206
- added C4: 100uF, rcl:C-USC1206
- added MDL1: (no value), ESP8266-ESP12E:ESP8266-12EESP8266-ESP12E
- added R10, R11, R12, R14, R8, R9: 10k, rcl:R-US_R0805
- R3, R6: value 10k -> 4.7k
- R4: value 4.7K -> 1k
Connections:
- net RELE1 renamed RELE
- removed net RELE2: U2.PC2(ADC2)
- removed net RFID_INT: JP1.5
- removed net RFID_MISO: JP1.4
- removed net RFID_MOSI: JP1.3
- removed net RFID_PW: U2.PD5(T1)
- removed net RFID_RST: JP1.7
- removed net RFID_SCK: JP1.2
- removed net RFID_SS: JP1.1
- removed net RFID_TX: U2.PD2(INT0)
- new net ESP_OC_NPROG: MDL1.GPIO0, R12.1
- new net ESP_OC_NRST: C15.1, MDL1.REST, R9.1
- new net ESP_RX_3V3: MDL1.RXD, U3.A5
- new net ESP_TX_3V3: MDL1.TXD, U3.A6
- new net LVLSHF_OC_OE: R14.1, U3.OE
- new net N$10: MDL1.CH_PD, R8.1
- new net N$13: MDL1.GPIO2, R11.1
- new net N$16: MDL1.GPIO15, R10.2
- new net N$8: U2.PB0(ICP), U3.B1
- new net RFID_MISO_3V3: JP1.4, U3.A4
- new net RFID_MOSI_3V3: JP1.3, U3.A3
- new net RFID_OC_NRST: JP1.7, U2.PD7(AIN1)
- new net RFID_SCK_3V3: JP1.2, U3.A2
- new net RFID_SS_3V3: JP1.1, U3.A1
- net +3V3: now also C13.1, C14.1, C4.1, MDL1.VCC, R11.2, R12.2, R14.2, R8.2, R9.2, U3.VCCA
- net +5V: now also C12.1, U3.VCCB
- net GND: now also C12.2, C13.2, C14.2, C15.2, C4.2, MDL1.GND, R10.1, U3.GND
- net N$17: now also U3.B2
- net N$18: now also U3.B4
- net N$19: now also U3.B3
- net N$21: now also U3.B6
- net N$22: now also U3.B5
Other:
- note added: "???"
- moved on the sheet: JP1, U3

Commit message: v2 esquematico semiterminado
Parts:
- added C16: 1000uF, rcl:CPOL-USE2.5-6
- added C17: 10uF, rcl:CPOL-USE2.5-6
- added D1: CD1206-S01575, diode:DIODE-MINIMELF
- added J2, J3: HDMI, partes v2:HDMI
- added JP2: M025MM, SparkFun-Connectors:M025MM
- added K1: (no value), pimoroni-mechanical:RELAY_EE2
- added Q3: PMBT3904, diego:PMBT3904
- added R15: 1k, rcl:R-US_R0805
- added R16: 10k, rcl:R-US_R0805
- added S1: (no value), SparkFun-Electromechanical:SWITCH-SPDTPTH
- added U1: ADP3338AKCZ-3.3RL7, ADI-Phase-2:ADP3338AKCZ-3.3RL7
Connections:
- new net HDMI_IN_5V: J3.+5V, K1.MAIN1, R16.1
- new net N$15: D1.A, K1.COIL-, Q3.C
- new net N$20: Q3.B, R15.2
- new net N$23: J2.TX2_N, J3.TX2_N
- new net N$24: J2.TX1_P, J3.TX1_P
- new net N$25: J2.TX1_N, J3.TX1_N
- new net N$26: J2.TX0_P, J3.TX0_P
- new net N$27: J2.TX0_N, J3.TX0_N
- new net N$28: J2.CLK_P, J3.CLK_P
- new net N$29: J2.CLK_N, J3.CLK_N
- new net N$30: J2.CEC_DAT, J3.CEC_DAT
- new net N$31: J2.SCL, J3.SCL
- new net N$32: J2.SDA, J3.SDA
- new net N$33: J2.HPD, J3.HPD
- new net N$34: R16.2, U2.PC2(ADC2)
- new net N$35: J2.+5V, K1.OFF1
- new net N$36: JP2.1, S1.P
- new net N$9: J2.TX2_P, J3.TX2_P
- net +3V3: now also C17.+, U1.OUT, U1.OUT_2
- net +5V: now also C16.+, D1.C, K1.COIL+, S1.O, U1.IN
- net GND: now also C16.-, C17.-, J2.GND@1, J2.GND@2, J2.GND@3, J2.GND@4, J2.GND@5, J2.GND@6, J2.GND@7, J2.GND@8, J2.GND@9, J3.GND@1, J3.GND@2, J3.GND@3, J3.GND@4, J3.GND@5, J3.GND@6, J3.GND@7, J3.GND@8, J3.GND@9, JP2.2, Q3.E, U1.GND
- net RELE: now also R15.1
