File: Hardware/pcb v2/sch y brd/pcb v2.sch (EAGLE design)
At the start: 53 parts, among them J1 AVR_SPI_PRG_6PTH, J2 HDMI, J3 HDMI, Q1 32.768kHz 12.5pF, Q2 PMBT3904, Q3 PMBT3904, U1 ADP3338AKCZ-3.3RL7, U2 ATMEGA328P, U3 TXS0108EPWR-TSSOP20, Y1 16Mhz

Commit message: fram
Parts:
- added C18: 100nF, rcl:C-USC0805
- added R17: 10k, rcl:R-US_R0805
- added U4: MB85RS16N, partes v2:MB85RS16N
Connections:
- net HDMI_IN_5V renamed HDMI_A_5V
- removed net N$35: J2.+5V, K1.OFF1
- new net HDMI_B_5V: J2.+5V, K1.OFF1, R17.1
- new net N$37: R17.2, U2.PC3(ADC3)
- new net N$39: U3.A7, U4.!CS
- new net N$40: U3.A8, U4.!HOLD
- net +3V3: now also C18.1, U4.VDD
- net GND: now also C18.2, U4.GND
- net RFID_MISO_3V3: now also U4.SO
- net RFID_MOSI_3V3: now also U4.SI
- net RFID_SCK_3V3: now also U4.SCK
Changed lines of the file:
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@@
 <?xml version="1.0" encoding="utf-8"?>
 <!DOCTYPE eagle SYSTEM "eagle.dtd">
-<eagle version="7.5.0">
+<eagle version="7.2.0">
 <drawing>
 <settings>
@@
 <part name="GND20" library="supply1" deviceset="GND" device=""/>
 <part name="GND21" library="supply1" deviceset="GND" device=""/>
+<part name="R17" library="rcl" deviceset="R-US_" device="R0805" value="10k"/>
+<part name="U4" library="partes v2" deviceset="MB85RS16N" device=""/>
+<part name="+3V3" library="supply1" deviceset="+3V3" device=""/>
+<part name="GND22" library="supply1" deviceset="GND" device=""/>
+<part name="C18" library="rcl" deviceset="C-US" device="C0805" value="100nF"/>
+<part name="GND23" library="supply1" deviceset="GND" device=""/>
 </parts>
 <sheets>
@@
 <plain>
 <text x="78.74" y="114.3" size="1.016" layer="97">???</text>
+<text x="238.76" y="-2.54" size="1.016" layer="97">???</text>
 </plain>
 <instances>
@@
 <instance part="GND20" gate="1" x="345.44" y="99.06"/>
 <instance part="GND21" gate="1" x="457.2" y="99.06"/>
+<instance part="R17" gate="G$1" x="144.78" y="78.74" rot="R180"/>
+<instance part="U4" gate="G$1" x="251.46" y="-2.54"/>
+<instance part="+3V3" gate="G$1" x="266.7" y="15.24" rot="MR0"/>
+<instance part="GND22" gate="1" x="238.76" y="-10.16"/>
+<instance part="C18" gate="G$1" x="279.4" y="5.08" rot="MR0"/>
+<instance part="GND23" gate="1" x="279.4" y="-5.08"/>
 </instances>
 <busses>
@@
 <pinref part="GND21" gate="1" pin="GND"/>
 </segment>
+<segment>
+<pinref part="C18" gate="G$1" pin="2"/>
+<pinref part="GND23" gate="1" pin="GND"/>
+<wire x1="279.4" y1="0" x2="279.4" y2="-2.54" width="0.1524" layer="91"/>
+</segment>
+<segment>
+<pinref part="GND22" gate="1" pin="GND"/>
+<pinref part="U4" gate="G$1" pin="GND"/>
+<wire x1="238.76" y1="-7.62" x2="238.76" y2="-5.08" width="0.1524" layer="91"/>
+<wire x1="238.76" y1="-5.08" x2="241.3" y2="-5.08" width="0.1524" layer="91"/>
+</segment>
 </net>
 <net name="+5V" class="0">
@@
 <segment>
 <pinref part="U3" gate="G$1" pin="A4"/>
-<wire x1="205.74" y1="20.32" x2="208.28" y2="20.32" width="0.1524" layer="91"/>
-<label x="208.28" y="20.32" size="1.016" layer="95" xref="yes"/>
+<wire x1="205.74" y1="20.32" x2="228.6" y2="20.32" width="0.1524" layer="91"/>
+<label x="231.14" y="20.32" size="1.016" layer="95" xref="yes"/>
+<pinref part="U4" gate="G$1" pin="SO"/>
+<wire x1="228.6" y1="20.32" x2="231.14" y2="20.32" width="0.1524" layer="91"/>
+<wire x1="241.3" y1="0" x2="228.6" y2="0" width="0.1524" layer="91"/>
+<wire x1="228.6" y1="0" x2="228.6" y2="20.32" width="0.1524" layer="91"/>
+<junction x="228.6" y="20.32"/>
 </segment>
 </net>
@@
 <segment>
 <pinref part="U3" gate="G$1" pin="A3"/>
-<wire x1="205.74" y1="22.86" x2="208.28" y2="22.86" width="0.1524" layer="91"/>
-<label x="208.28" y="22.86" size="1.016" layer="95" xref="yes"/>
+<wire x1="205.74" y1="22.86" x2="226.06" y2="22.86" width="0.1524" layer="91"/>
+<label x="231.14" y="22.86" size="1.016" layer="95" xref="yes"/>
+<pinref part="U4" gate="G$1" pin="SI"/>
+<wire x1="226.06" y1="22.86" x2="231.14" y2="22.86" width="0.1524" layer="91"/>
+<wire x1="264.16" y1="-5.08" x2="266.7" y2="-5.08" width="0.1524" layer="91"/>
+<wire x1="266.7" y1="-5.08" x2="266.7" y2="-15.24" width="0.1524" layer="91"/>
+<wire x1="266.7" y1="-15.24" x2="226.06" y2="-15.24" width="0.1524" layer="91"/>
+<wire x1="226.06" y1="-15.24" x2="226.06" y2="22.86" width="0.1524" layer="91"/>
+<junction x="226.06" y="22.86"/>
 </segment>
 </net>
@@
 <segment>
 <pinref part="U3" gate="G$1" pin="A2"/>
-<wire x1="205.74" y1="25.4" x2="208.28" y2="25.4" width="0.1524" layer="91"/>
-<label x="208.28" y="25.4" size="1.016" layer="95" xref="yes"/>
+<wire x1="205.74" y1="25.4" x2="223.52" y2="25.4" width="0.1524" layer="91"/>
+<label x="231.14" y="25.4" size="1.016" layer="95" xref="yes"/>
+<pinref part="U4" gate="G$1" pin="SCK"/>
+<wire x1="223.52" y1="25.4" x2="231.14" y2="25.4" width="0.1524" layer="91"/>
+<wire x1="264.16" y1="-2.54" x2="269.24" y2="-2.54" width="0.1524" layer="91"/>
+<wire x1="269.24" y1="-2.54" x2="269.24" y2="-17.78" width="0.1524" layer="91"/>
+<wire x1="269.24" y1="-17.78" x2="223.52" y2="-17.78" width="0.1524" layer="91"/>
+<wire x1="223.52" y1="-17.78" x2="223.52" y2="25.4" width="0.1524" layer="91"/>
+<junction x="223.52" y="25.4"/>
 </segment>
 </net>
@@
 <segment>
 <pinref part="U3" gate="G$1" pin="A1"/>
-<wire x1="205.74" y1="27.94" x2="208.28" y2="27.94" width="0.1524" layer="91"/>
-<label x="208.28" y="27.94" size="1.016" layer="95" xref="yes"/>
+<wire x1="205.74" y1="27.94" x2="231.14" y2="27.94" width="0.1524" layer="91"/>
+<label x="231.14" y="27.94" size="1.016" layer="95" xref="yes"/>
 </segment>
 </net>
@@
 <pinref part="C17" gate="G$1" pin="+"/>
 </segment>
+<segment>
+<pinref part="+3V3" gate="G$1" pin="+3V3"/>
+<wire x1="266.7" y1="12.7" x2="266.7" y2="10.16" width="0.1524" layer="91"/>
+<wire x1="266.7" y1="10.16" x2="279.4" y2="10.16" width="0.1524" layer="91"/>
+<pinref part="C18" gate="G$1" pin="1"/>
+<wire x1="279.4" y1="10.16" x2="279.4" y2="7.62" width="0.1524" layer="91"/>
+<pinref part="U4" gate="G$1" pin="VDD"/>
+<wire x1="266.7" y1="10.16" x2="266.7" y2="2.54" width="0.1524" layer="91"/>
+<wire x1="266.7" y1="2.54" x2="264.16" y2="2.54" width="0.1524" layer="91"/>
+<junction x="266.7" y="10.16"/>
+</segment>
 </net>
 <net name="N$7" class="0">
@@
 </segment>
 </net>
-<net name="HDMI_IN_5V" class="0">
+<net name="HDMI_A_5V" class="0">
 <segment>
 <pinref part="J3" gate="G$1" pin="+5V"/>
@@
 </segment>
 </net>
-<net name="N$35" class="0">
+<net name="HDMI_B_5V" class="0">
 <segment>
 <pinref part="K1" gate="G$1" pin="OFF1"/>
@@
 <pinref part="J2" gate="G$1" pin="+5V"/>
 <wire x1="459.74" y1="78.74" x2="449.58" y2="78.74" width="0.1524" layer="91"/>
+<wire x1="459.74" y1="78.74" x2="467.36" y2="78.74" width="0.1524" layer="91"/>
+<junction x="459.74" y="78.74"/>
+<label x="467.36" y="78.74" size="1.016" layer="95" xref="yes"/>
+</segment>
+<segment>
+<pinref part="R17" gate="G$1" pin="1"/>
+<wire x1="149.86" y1="78.74" x2="157.48" y2="78.74" width="0.1524" layer="91"/>
+<label x="157.48" y="78.74" size="1.016" layer="95" xref="yes"/>
 </segment>
 </net>
@@
 </segment>
 </net>
+<net name="N$37" class="0">
+<segment>
+<pinref part="U2" gate="G$1" pin="PC3(ADC3)"/>
+<wire x1="116.84" y1="83.82" x2="137.16" y2="83.82" width="0.1524" layer="91"/>
+<wire x1="137.16" y1="83.82" x2="137.16" y2="78.74" width="0.1524" layer="91"/>
+<pinref part="R17" gate="G$1" pin="2"/>
+<wire x1="137.16" y1="78.74" x2="139.7" y2="78.74" width="0.1524" layer="91"/>
+</segment>
+</net>
+<net name="N$39" class="0">
+<segment>
+<pinref part="U4" gate="G$1" pin="!CS"/>
+<wire x1="241.3" y1="2.54" x2="231.14" y2="2.54" width="0.1524" layer="91"/>
+<wire x1="231.14" y1="2.54" x2="231.14" y2="12.7" width="0.1524" layer="91"/>
+<pinref part="U3" gate="G$1" pin="A7"/>
+<wire x1="231.14" y1="12.7" x2="205.74" y2="12.7" width="0.1524" layer="91"/>
+</segment>
+</net>
+<net name="N$40" class="0">
+<segment>
+<pinref part="U4" gate="G$1" pin="!HOLD"/>
+<wire x1="264.16" y1="0" x2="271.78" y2="0" width="0.1524" layer="91"/>
+<wire x1="271.78" y1="0" x2="271.78" y2="-20.32" width="0.1524" layer="91"/>
+<wire x1="271.78" y1="-20.32" x2="220.98" y2="-20.32" width="0.1524" layer="91"/>
+<wire x1="220.98" y1="-20.32" x2="220.98" y2="10.16" width="0.1524" layer="91"/>
+<pinref part="U3" gate="G$1" pin="A8"/>
+<wire x1="220.98" y1="10.16" x2="205.74" y2="10.16" width="0.1524" layer="91"/>
+</segment>
+</net>

Commit message: v2 esquematico completo
Parts:
- removed U$1: DS1307SO8, SparkFun-FreqCtrl:DS1307SO8
- added C19: 1uF, rcl:C-USC0805
- added C20: 100nF, rcl:C-USC0805
- added J4: HDMI, partes v2:HDMI
- added JP3: (no value), SparkFun-Connectors:M081X08
- added JP4: 2X6 FEMALE, SparkFun-Connectors:M06X2PTH_FEMALE
- added U5: DS1307SO8, SparkFun-FreqCtrl:DS1307SO8
- C10: value 100nF -> 10uF; device rcl:C-USC0805 -> rcl:C-USC1206
- C11: device rcl:C-USC0805 -> rcl:C-USC1206
- C15: value 470pF -> 10uF; device rcl:C-USC1206 -> rcl:CPOL-USE2.5-6
- C17: value 10uF -> 100nF; device rcl:CPOL-USE2.5-6 -> rcl:C-USC0805
- C18: value 100nF -> 10uF; device rcl:C-USC0805 -> rcl:CPOL-USE2.5-6
- C4: value 100uF -> 100nF; device rcl:C-USC1206 -> rcl:C-USC0805
- C5, C6: value 100nF -> 22pF; device rcl:C-USC0805 -> rcl:C-USC1206
- C7: value 22pF -> 100nF; device rcl:C-USC1206 -> rcl:C-USC0805
- C8: value 22pF -> 470pF
- C9: value 100nF -> 100uF; device rcl:C-USC0805 -> rcl:C-USC1206
- J2: value HDMI -> 1981584-1; device partes v2:HDMI -> con-usb:1981584-1; MF (none) -> Hirose; MPN (none) -> ZX62-AB-5PA(11)
- JP1: device SparkFun-Connectors:M081X08 -> SparkFun-Connectors:M03JST-SMD
- JP2: value M025MM -> FEMALE 2x3; device SparkFun-Connectors:M025MM -> SparkFun-Connectors:M03X2FEMALE
- Q1: value 32.768kHz 12.5pF -> PMBT3904; device crystal:CRYSTALTC26H -> diego:PMBT3904
- Q3: value PMBT3904 -> 32.768kHz 12.5pF; device diego:PMBT3904 -> crystal:CRYSTALTC26H
- R1: value 1K -> NO(10k)
- R10: value 10k -> 0
- R12, R9: value 10k -> 1k
- R13: value 10K -> 1K
- R15, R4: value 1k -> 10k
- R16, R17: value 10k -> 4.7k
- R3, R6: value 4.7k -> 10k
- R5: value 1K -> 10k
- R7: value 0 -> 10k
- S1: value (none) -> SWITCH-MOMENTARY-2SMD; device SparkFun-Electromechanical:SWITCH-SPDTPTH -> SparkFun-Electromechanical:SWITCH-MOMENTARY-2SMD
- U1: value ADP3338AKCZ-3.3RL7 -> ATMEGA328P; device ADI-Phase-2:ADP3338AKCZ-3.3RL7 -> SparkFun-DigitalIC:ATMEGA328_SMT
- U2: value ATMEGA328P -> TXS0108EPWR-TSSOP20; device SparkFun-DigitalIC:ATMEGA328_SMT -> Seeed-IC-2016:LOGIC-TXS0108EPWR(TSSOP20)
- U3: value TXS0108EPWR-TSSOP20 -> MB85RS16N; device Seeed-IC-2016:LOGIC-TXS0108EPWR(TSSOP20) -> partes v2:MB85RS16N
- U4: value MB85RS16N -> ADP3338AKCZ-3.3RL7; device partes v2:MB85RS16N -> ADI-Phase-2:ADP3338AKCZ-3.3RL7
Connections:
- removed net N$36: JP2.1, S1.P
- removed net N$40: U3.A8, U4.!HOLD
- removed net RST_ATM_FLANCO: C9.1, R1.2
- new net ADC6: JP4.3, U1.ADC6
- new net ADC7: JP4.5, U1.ADC7
- new net BOTON: R15.1, S1.1, U1.PD2(INT0)
- new net N$41: U1.PD6(AIN0), U2.B7
- new net PB2: JP4.6, U1.PB2(SS/OC1B)
- new net PD3: JP4.7, U1.PD3(INT1)
- new net PD4: JP4.9, U1.PD4(XCK/T0)
- new net PD5: JP4.4, U1.PD5(T1)
- new net RST_ATM_3V3: MDL1.GPIO4, U2.A8
- net +3V3: now also C10.1, C11.1, C12.1, C17.1, C18.+, C9.1, JP3.8, JP4.2, R2.2, R4.2, R5.2, R6.2, U2.VCCA, U3.!HOLD, U3.!WP, U3.VDD, U4.OUT, U4.OUT_2; no longer C13.1, C17.+, C18.1, C4.1, JP1.8, R12.2, R14.2, R8.2, R9.2, U1.OUT, U1.OUT_2, U3.VCCA, U4.VDD
- net +5V: now also C1.1, C13.1, C15.+, C19.1, C20.1, J2.VBUS, JP1.3, JP4.1, R1.2, R13.2, R14.2, R15.2, R16.2, R17.2, U1.AVCC, U1.VCC@1, U1.VCC@2, U2.VCCB, U4.IN, U5.VCC; no longer C10.1, C11.1, C12.1, C5.1, R13.1, R2.2, R3.2, R5.2, R6.2, S1.O, U$1.VCC, U1.IN, U2.AVCC, U2.VCC@1, U2.VCC@2, U3.VCCB
- net BUZZER: now also R12.1, U1.PC0(ADC0); no longer R4.1, U2.PC0(ADC0)
- net ESP_OC_NPROG: now also JP2.5, R2.1; no longer R12.1
- net ESP_OC_NRST: now also C8.1, JP2.4, R6.1; no longer C15.1, R9.1
- net ESP_RX_3V3: now also JP2.1, U2.A5; no longer U3.A5
- net ESP_TX_3V3: now also JP2.2, U2.A6; no longer U3.A6
- net GND: now also C15.-, C17.2, C18.-, C19.2, C20.2, C9.2, J2.GND, J2.S1, J2.S2, J2.S3, J2.S4, J4.GND@1, J4.GND@2, J4.GND@3, J4.GND@4, J4.GND@5, J4.GND@6, J4.GND@7, J4.GND@8, J4.GND@9, JP1.1, JP3.6, JP4.11, JP4.12, Q1.E, R3.1, S1.2, U1.AGND, U1.GND@1, U1.GND@2, U2.GND, U5.GND; no longer C15.2, C17.-, C18.2, J2.GND@1, J2.GND@2, J2.GND@3, J2.GND@4, J2.GND@5, J2.GND@6, J2.GND@7, J2.GND@8, J2.GND@9, JP1.6, JP2.2, Q3.E, R1.1, R10.1, U$1.GND, U1.GND, U2.AGND, U2.GND@1, U2.GND@2
- net HDMI_A_5V: now also R7.1; no longer R16.1
- net HDMI_B_5V: now also J4.+5V, R8.1; no longer J2.+5V, R17.1
- net LED: now also JP1.2, U1.PB1(OC1A); no longer U2.PB1(OC1A)
- net LVLSHF_OC_OE: now also JP2.3, R11.1, U2.OE; no longer R14.1, U3.OE
- net N$1: now also R12.2; no longer R4.2
- net N$10: now also R5.1; no longer R8.1
- net N$11: now also C5.1, U1.PB6(XTAL1/TOSC1); no longer C7.1, U2.PB6(XTAL1/TOSC1)
- net N$12: now also C6.1, U1.PB7(XTAL2/TOSC2); no longer C8.1, U2.PB7(XTAL2/TOSC2)
- net N$13: now also R4.1; no longer R11.1
- net N$14: now also C4.1, U1.AREF; no longer C6.1, U2.AREF
- net N$15: now also D2.A, Q1.C; no longer D1.A, Q3.C
- net N$16: now also R3.2; no longer R10.2
- net N$17: now also U1.PB5(SCK), U2.B2; no longer U2.PB5(SCK), U3.B2
- net N$18: now also U1.PB4(MISO), U2.B4; no longer U2.PB4(MISO), U3.B4
- net N$19: now also U1.PB3(MOSI/OC2), U2.B3; no longer U2.PB3(MOSI/OC2), U3.B3
- net N$2: now also Q3.2, U5.X1; no longer Q1.2, U$1.X1
- net N$20: now also Q1.B, R9.2; no longer Q3.B, R15.2
- net N$21: now also U1.PD0(RXD), U2.B6; no longer U2.PD0(RXD), U3.B6
- net N$22: now also U1.PD1(TXD), U2.B5; no longer U2.PD1(TXD), U3.B5
- net N$23: now also J4.TX2_N; no longer J2.TX2_N
- net N$24: now also J4.TX1_P; no longer J2.TX1_P
- net N$25: now also J4.TX1_N; no longer J2.TX1_N
- net N$26: now also J4.TX0_P; no longer J2.TX0_P
- net N$27: now also J4.TX0_N; no longer J2.TX0_N
- net N$28: now also J4.CLK_P; no longer J2.CLK_P
- net N$29: now also J4.CLK_N; no longer J2.CLK_N
- net N$3: now also Q3.1, U5.X2; no longer Q1.1, U$1.X2
- net N$30: now also J4.CEC_DAT; no longer J2.CEC_DAT
- net N$31: now also J4.SCL; no longer J2.SCL
- net N$32: now also J4.SDA; no longer J2.SDA
- net N$33: now also J4.HPD; no longer J2.HPD
- net N$34: now also R7.2, U1.PC2(ADC2); no longer R16.2, U2.PC2(ADC2)
- net N$37: now also R8.2, U1.PC3(ADC3); no longer R17.2, U2.PC3(ADC3)
- net N$39: now also U2.A7, U3.!CS; no longer U3.A7, U4.!CS
- net N$4: now also U5.VBATT; no longer U$1.VBATT
- net N$5: now also R13.1; no longer R5.1
- net N$6: now also R14.1, U5.SQW; no longer R2.1, U$1.SQW
- net N$7: now also R10.1, U2.B8; no longer C9.2, R7.2
- net N$8: now also U1.PB0(ICP), U2.B1; no longer U2.PB0(ICP), U3.B1
- net N$9: now also J4.TX2_P; no longer J2.TX2_P
- net RELE: now also R9.1, U1.PC1(ADC1); no longer R15.1, U2.PC1(ADC1)
- net RFID_MISO_3V3: now also JP3.4, U2.A4, U3.SO; no longer JP1.4, U3.A4, U4.SO
- net RFID_MOSI_3V3: now also JP3.3, U2.A3, U3.SI; no longer JP1.3, U3.A3, U4.SI
- net RFID_OC_NRST: now also JP3.7, U1.PD7(AIN1); no longer JP1.7, U2.PD7(AIN1)
- net RFID_SCK_3V3: now also JP3.2, U2.A2, U3.SCK; no longer JP1.2, U3.A2, U4.SCK
- net RFID_SS_3V3: now also JP3.1, U2.A1; no longer JP1.1, U3.A1
- net RST_ATM: now also C7.1, D1.A, R1.1, R10.2, U1.PC6(/RESET); no longer C1.1, D2.A, R13.2, R7.1, U2.PC6(/RESET)
- net SCL: now also JP4.10, R16.1, U1.PC5(ADC5/SCL), U5.SCL; no longer R3.1, U$1.SCL, U2.PC5(ADC5/SCL)
- net SDA: now also JP4.8, R17.1, U1.PC4(ADC4/SDA), U5.SDA; no longer R6.1, U$1.SDA, U2.PC4(ADC4/SDA)
Other:
- note removed: "???"
- moved on the sheet: C1, C10, C11, C12, C13, C14, C16, C3, C4, C5, C6, C7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
