File: Hardware/pcb v3/sch y brd/pcb v3.brd (EAGLE design)
At the start: 80 x 80 mm, 43 parts, among them J2 1981584-1, J3 HDMI, J4 JST-3, J5 HDMI, J6 FEMALE 2x3, Q1 PMBT3904, Q2 PMBT3904, U1 NCP1117LPST33T3G, U2 MCP79510, U4 DS1307SO8, Y1 CRYSTAL.ABS25, Y2 MC-306

Commit message: rtc y led V3
Parts:
- removed BAT1: BK-885, SparkFun-Electromechanical:BATTCON_12MM
- removed BT1: 1225BAT, partes v2:BHSD-1225-SM
- removed R16, R17: 4.7k, rcl:R0603
- removed U4: DS1307SO8, SparkFun-FreqCtrl:SO08
- removed Y2: MC-306, crystal:MC-306
- added BAT2: BAT-HLD-001, battery:BATTCON_20MM
- added C2: 18pF, rcl:C0805
- added C3: 100pF, rcl:C0805
- added C4: 100nF, rcl:C0805
- added D1: DB2S311, adafruit:SOD-523
- added Q3: BSS138, SparkFun-DiscreteSemi:SOT23-3
- added R1: 1k, rcl:R0805
- added R7: 10k, rcl:R0805
- added U3: 74HCT1G125GW, NXP_By_element14_Batch_1:SOT65P210X110-5N
- C18: device rcl:C0603 -> rcl:C0805
Connections:
- removed net +: BAT1.PWR@1
- removed net -: BAT1.GND
- removed net ESP_GPIO13_3V3: MDL1.7
- removed net LED: J4.2
- removed net SCL: R16.1, U4.6
- removed net SDA: R17.1, U4.5
- new net LED/RX: MDL1.15, U3.2
- new net MISO: MDL1.6, U2.7
- new net MOSI: MDL1.7, U2.6
- new net N$11: J4.2, U3.4
- new net N$4: R7.2, U3.1
- new net N$7: BAT2.1, D1.A
- new net N$8: D1.K, R1.2
- new net RTC_!CS: U2.4
- new net SCK: MDL1.5, U2.8
- new net TX: MDL1.16
- net +3V3: now also C18.1, R14.2, U2.10
- net +5V: now also C4.1, U3.5; no longer C18.1, R14.2, R16.2, R17.2, U4.8
- net BOTON: no longer MDL1.5
- net ESP_RX_3V3: no longer MDL1.15
- net ESP_TX_3V3: no longer MDL1.16
- net GND: now also BAT2.2, C1.2, C2.2, C3.2, C4.2, R7.1, U2.5, U3.3; no longer BT1.V-, U4.4
- net N$2: now also C1.1, U2.1, Y1.4; no longer U4.1, Y2.4
- net N$3: now also C2.1, U2.2, Y1.1; no longer U4.2, Y2.1
- net N$6: now also U2.9; no longer U4.7
- net N$9: now also C3.1, R1.1, U2.3; no longer BT1.V+, U4.3
Routing:
- net SDA: track 85.5 -> 0.00 mm, vias 4 -> 0
- net SCL: track 82.7 -> 0.00 mm, vias 4 -> 0
- net LED: track 48.7 -> 0.00 mm, vias 3 -> 0
- net MOSI: track 0.00 -> 21.1 mm, vias 0 -> 4
- net ESP_GPIO13_3V3: track 21.1 -> 0.00 mm, vias 4 -> 0
- net +5V: track 260.4 -> 248.3 mm
- net N$9: track 8.19 -> 0.00 mm, vias 1 -> 0
- net N$2: track 7.74 -> 0.00 mm
- net N$3: track 6.56 -> 0.00 mm
- net +3V3: track 137.0 -> 141.6 mm
- net ESP_RX_3V3: track 107.9 -> 104.4 mm
- net ESP_TX_3V3: track 115.4 -> 112.0 mm
- net BOTON: track 122.0 -> 119.7 mm
- net N$6: track 4.04 -> 1.80 mm

Commit message: esquematico y bom v3 completo
Parts:
- removed C16: 10uF, rcl:UD-5X5,8_NICHICON
- removed C17: 1uF, rcl:C0805
- removed C18: 100nF, rcl:C0805
- removed D2: CD1206-S01575, diode:MINIMELF
- removed J5: HDMI, partes v2:0471511071
- removed J6: FEMALE 2x3, SparkFun-Connectors:2X3
- removed K1: (no value), pimoroni-mechanical:RELAY-EE2
- removed Q2: PMBT3904, diego:SOT-23-3
- removed Q3: BSS138, SparkFun-DiscreteSemi:SOT23-3
- removed R15: 10k, rcl:R0603
- added C12: 10uF, rcl:C0805
- added C5: 100nF, rcl:C0805
- added J1: JST-3, partes v2:B3B-PH-SM4-TB
- added JP1: (no value), SparkFun-Connectors:1X08
- added R10, R8: 10k, rcl:R0805
- added R11: 1k, rcl:R0805
- added U4: 74HCT1G125GW, NXP_By_element14_Batch_1:SOT65P210X110-5N
- added U5: NCP1117LPST33T3G, SparkFun-PowerIC:SOT223
- C1: value 18pF -> 100nF
- C10: device rcl:C0603 -> rcl:C0805
- C2: value 18pF -> 100pF
- C3: value 100pF -> 18pF
- C4: value 100nF -> 18pF
- C6: value 470pF -> 100uF; device rcl:C0603 -> rcl:C1206
- C7: value 100uF -> 100nF; device rcl:C1206 -> rcl:C0805
- C8: value 10uF -> 100nF
- C9: value 1uF -> 100nF
- J2: value 1981584-1 -> HDMI; device con-usb:1981584-1 -> partes v2:0471511071
- J4: value JST-3 -> 1981584-1; device partes v2:B3B-PH-SM4-TB -> con-usb:1981584-1
- R1, R13, R9: value 1k -> 10k
- R14: value 10k -> 27k; device rcl:R0603 -> rcl:R0805
- R2, R3, R4, R6: device rcl:R0603 -> rcl:R0805
- R5: value 10k -> 1k; device rcl:R0603 -> rcl:R0805
- U1: value NCP1117LPST33T3G -> 74HCT1G125GW; device SparkFun-PowerIC:SOT223 -> NXP_By_element14_Batch_1:SOT65P210X110-5N
- U3: value 74HCT1G125GW -> MC74VHC1GT66; device NXP_By_element14_Batch_1:SOT65P210X110-5N -> hoky:TSOP-5
- moved R9 210.0 mm to (-22.9, -147.3), flipped to the top, turned to 0 degrees
- moved R14 196.4 mm to (-22.9, -158.8)
- moved R13 186.2 mm to (-22.9, -111.1), turned to 0 degrees
- moved C9 171.9 mm to (-22.9, -141.0), flipped to the top, turned to 0 degrees
- moved C8 124.1 mm to (-22.9, -92.1), flipped to the top, turned to 0 degrees
- moved R4 96.0 mm to (-22.9, -69.8), flipped to the top, turned to 0 degrees
- moved R7 92.0 mm to (17.8, 12.7), flipped to the bottom
- moved J4 89.5 mm to (14.6, 80.0), flipped to the top
- moved R5 71.8 mm to (-19.1, -47.0), flipped to the top
- moved R1 65.9 mm to (10.2, 12.1), flipped to the bottom, turned to 270 degrees
- moved Q1 60.8 mm to (5.08, 72.4), flipped to the top, turned to 0 degrees
- moved U1 60.3 mm to (-19.7, -62.2)
- moved C7 60.2 mm to (71.8, 15.2), flipped to the top, turned to 180 degrees
- moved C1 57.3 mm to (-22.9, -76.2)
- moved C10 52.2 mm to (8.26, 76.8), flipped to the top
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- renumbered BAT2 to BAT1, C14 to C11
Connections:
- removed net ESP_OC_NPROG: J6.5, MDL1.12, R2.1
- removed net ESP_OC_NRST: C6.1, J6.4, MDL1.1, R6.1
- removed net ESP_RX_3V3: J6.1
- removed net ESP_TX_3V3: J6.2
- removed net HDMI_A_5V: J3.P$18, K1.4
- removed net HDMI_B_5V: J5.P$18, K1.5
- removed net LVLSHF_OC_OE: J6.3
- removed net N$13: MDL1.11, R4.1
- removed net N$20: Q1.1, R9.2
- removed net RELE: R9.1
- removed net RFID_MISO_3V3: A1.MISO
- removed net RFID_MOSI_3V3: A1.MOSI
- removed net RFID_OC_NRST: A1.RST
- removed net RFID_SCK_3V3: A1.SCK
- removed net RFID_SS_3V3: A1.SDA
- removed net RST_ATM_3V3: MDL1.13
- removed net RTC_!CS: U2.4
- new net !RST: C5.1, JP1.6, MDL1.1, R7.1
- new net HDMI_IN_5V: J2.P$18, MDL1.14, R9.2, U3.1
- new net HDMI_OUT_5V: J3.P$18, JP1.1, U3.2, U4.4
- new net HDMI_SW: MDL1.10, R2.2, U3.4, U4.2
- new net PROG/RTC_!CS: JP1.7, MDL1.12, R1.1, U2.4
- new net RFID_!CS: A1.SDA, MDL1.11, R3.1
- net +3V3: now also C13.1, C6.1, JP1.3, R1.2, R3.2, R7.2, R8.2, S1.P$1, U5.2, U5.4; no longer C10.1, C16.+, C18.1, C8.1, C9.1, R14.2, R15.2, R2.2, R4.2, R5.2, U1.2, U1.4
- net +5V: now also C1.1, C10.1, C12.1, C8.1, C9.1, J1.3, J4.1, JP1.2, R12.2, U1.5, U4.5, U5.3; no longer C13.1, C17.1, C4.1, D2.C, J2.1, J4.3, K1.1, R13.2, U1.3
- net BOTON: now also MDL1.2, R13.2, R14.1; no longer R15.1, S1.P$1
- net BUZZER: now also MDL1.13, R11.1; no longer R12.1
- net CLK_N: now also J2.P$12; no longer J5.P$12
- net CLK_P: now also J2.P$10; no longer J5.P$10
- net GND: now also C12.2, C5.2, J1.1, J2.P$11, J2.P$17, J2.P$2, J2.P$20, J2.P$21, J2.P$22, J2.P$23, J2.P$5, J2.P$8, J4.5, J4.S1, J4.S2, J4.S3, J4.S4, JP1.8, R10.1, R13.1, R2.1, R4.1, R9.1, U1.3, U4.3, U5.1; no longer C16.-, C17.2, C18.2, J2.5, J2.S1, J2.S2, J2.S3, J2.S4, J4.1, J5.P$11, J5.P$17, J5.P$2, J5.P$20, J5.P$21, J5.P$22, J5.P$23, J5.P$5, J5.P$8, J6.6, Q2.2, R3.1, R7.1, S1.P$3, S1.P$4, U1.1
- net LED/RX: now also JP1.4, U1.2; no longer U3.2
- net MISO: now also A1.MISO
- net MOSI: now also A1.MOSI
- net N$1: now also Q1.1, R11.2; no longer Q2.1, R12.2
- net N$10: now also R6.1; no longer R5.1
- net N$11: now also J1.2, U1.4; no longer J4.2, U3.4
- net N$15: now also R10.2, U4.1; no longer D2.A, K1.12, Q1.3
- net N$16: now also S1.P$3, S1.P$4; no longer MDL1.10, R3.2
- net N$2: now also C3.1; no longer C1.1
- net N$3: now also C4.1; no longer C2.1
- net N$30: now also J2.P$13; no longer J5.P$13
- net N$31: now also J2.P$15; no longer J5.P$15
- net N$32: now also J2.P$16; no longer J5.P$16
- net N$33: now also J2.P$19; no longer J5.P$19
- net N$4: now also R4.2, U1.1; no longer R7.2, U3.1
- net N$5: now also Q1.3, R12.1; no longer Q2.3, R13.1
- net N$6: now also R8.1; no longer R14.1
- net N$8: now also R5.2; no longer R1.2
- net N$9: now also C2.1, R5.1; no longer C3.1, R1.1
- net SCK: now also A1.SCK
- net TX: now also JP1.5
- net TX0_N: now also J2.P$9; no longer J5.P$9
- net TX0_P: now also J2.P$7; no longer J5.P$7
- net TX1_N: now also J2.P$6; no longer J5.P$6
- net TX1_P: now also J2.P$4; no longer J5.P$4
- net TX2_N: now also J2.P$3; no longer J5.P$3
- net TX2_P: now also J2.P$1; no longer J5.P$1
Routing:
- net BOTON: track 119.7 -> 0.00 mm, vias 8 -> 0
- net ESP_TX_3V3: track 112.0 -> 0.00 mm, vias 5 -> 0
- net ESP_RX_3V3: track 104.4 -> 0.00 mm, vias 5 -> 0
- net ESP_OC_NPROG: track 101.3 -> 0.00 mm, vias 5 -> 0
- net PROG/RTC_!CS: track 0.00 -> 100.6 mm, vias 0 -> 5
- net ESP_OC_NRST: track 87.4 -> 0.00 mm, vias 4 -> 0
- net HDMI_A_5V: track 85.6 -> 0.00 mm, vias 4 -> 0
- net !RST: track 0.00 -> 85.4 mm, vias 0 -> 4
- net HDMI_IN_5V: track 0.00 -> 82.7 mm, vias 0 -> 4
- net RELE: track 69.8 -> 0.00 mm, vias 5 -> 0
- net LVLSHF_OC_OE: track 63.3 -> 0.00 mm, vias 4 -> 0
- net RFID_OC_NRST: track 62.2 -> 0.00 mm, vias 5 -> 0
- net +3V3: track 141.6 -> 97.3 mm, vias 39 -> 36
- net BUZZER: track 76.7 -> 117.0 mm, vias 7 -> 9
- net RST_ATM_3V3: track 40.3 -> 0.00 mm, vias 2 -> 0
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
Commit message: Ruteo pcb V3 completo
Parts:
- C11: value 1200uF -> 100uF; device rcl:UD-10X10_NICHICON -> rcl:UD-6,3X5,8_NICHICON
- R13: value 10k -> 27k
- R14: value 27k -> 10k
- moved R9 198.0 mm to (67.9, 28.6), turned to 90 degrees
- moved R14 193.8 mm to (41.3, 24.1), turned to 270 degrees
- moved JP1 193.7 mm to (77.5, 11.4), turned to 90 degrees
- moved C9 188.6 mm to (58.4, 29.2)
- moved R10 187.7 mm to (65.4, 28.6), turned to 90 degrees
- moved U4 181.2 mm to (62.2, 28.6), turned to 90 degrees
- moved C12 159.0 mm to (6.99, 32.4)
- moved C8 151.1 mm to (61.0, 33.7)
- moved U3 146.7 mm to (65.4, 33.7)
- moved R13 146.3 mm to (42.5, 19.7)
- moved C1 91.4 mm to (8.89, 9.53), turned to 180 degrees
- moved R4 90.1 mm to (11.7, 13.3)
- moved C2 85.1 mm to (43.2, 4.76), turned to 90 degrees
- moved R5 82.9 mm to (45.7, 4.76), turned to 90 degrees
- moved U1 79.3 mm to (12.7, 10.2), turned to 90 degrees
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Connections:
- removed net N$16: S1.P$3, S1.P$4
- new net N$12: R13.2, S1.P$3, S1.P$4
- net BOTON: now also R13.1, R14.2; no longer R13.2, R14.1
- net GND: now also JP1.1, R14.1; no longer JP1.8, R13.1
- net HDMI_OUT_5V: now also JP1.8; no longer JP1.1
- net N$2: now also Y1.1; no longer Y1.4
- net N$3: now also Y1.4; no longer Y1.1
Routing:
- net +3V3: track 97.3 -> 268.2 mm
- net LED/RX: track 0.00 -> 78.3 mm, vias 0 -> 2
- net TX: track 0.00 -> 76.5 mm, vias 0 -> 2
- net BUZZER: track 117.0 -> 41.0 mm, vias 9 -> 2
- net HDMI_SW: track 2.86 -> 71.7 mm
- net N$12: track 0.00 -> 57.8 mm
- net N$33: track 91.7 -> 39.3 mm, vias 0 -> 2
- net MISO: track 3.88 -> 55.3 mm, vias 0 -> 2
- net SCK: track 11.1 -> 60.4 mm, vias 1 -> 3
- net N$32: track 82.2 -> 37.3 mm, vias 0 -> 2
- net N$31: track 77.6 -> 40.3 mm, vias 0 -> 2
- net +5V: track 210.4 -> 247.3 mm, vias 12 -> 2
- net MOSI: track 27.8 -> 61.4 mm, vias 5 -> 4
- net N$7: track 0.00 -> 32.2 mm
- net N$30: track 72.3 -> 40.7 mm, vias 0 -> 2
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Other:
- board size 80 x 80 mm -> 80 x 50 mm
- board text added: "20-07-16"
- board text added: "CR20XX"
- board text added: "Hoky V3"
- board text removed: "Hoky V2r1 01-07-16"

Commit message: gerbers v3
Parts:
- added R15, R16: 10k, rcl:R0805
- C11: device rcl:UD-6,3X5,8_NICHICON -> hoky:UD-6,3X5,8_NICHICON_LPADS
- R13: value 27k -> 10k
- moved R13 0.90 mm to (43.2, 20.3)
- moved C3 0.32 mm to (43.2, 7.94)
- moved C7 0.32 mm to (44.1, 1.59)
- moved C11 0.32 mm to (5.40, 38.1)
Connections:
- new net N$13: R13.1, R15.2
- new net N$14: R15.1, R16.2
- net BOTON: now also R16.1; no longer R13.1
Routing:
- net N$13: track 0.00 -> 5.87 mm
- net BOTON: track 20.3 -> 24.6 mm
- net N$14: track 0.00 -> 2.54 mm
- net +5V: track 247.3 -> 248.6 mm
- net +3V3: track 268.2 -> 268.7 mm
- net GND: vias 104 -> 106
