File: Hardware/pcb v3/sch y brd/pcb v3.sch (EAGLE design)
At the start: 43 parts, among them J2 1981584-1, J3 HDMI, J4 JST-3, J5 HDMI, J6 FEMALE 2x3, Q1 PMBT3904, Q2 PMBT3904, U1 NCP1117LPST33T3G, U2 MCP79510, U4 DS1307SO8, Y1 CRYSTAL.ABS25, Y2 MC-306

Commit message: rtc y led V3
Parts:
- removed BAT1: BK-885, SparkFun-Electromechanical:BATTERY12MM
- removed BT1: 1225BAT, partes v2:1225BAT
- removed R16, R17: 4.7k, rcl:R-US_R0603
- removed U4: DS1307SO8, SparkFun-FreqCtrl:DS1307SO8
- removed Y2: MC-306, crystal:MC-306
- added BAT2: BAT-HLD-001, battery:LINX-BAT-HLD-00120SMD
- added C2: 18pF, rcl:C-USC0805
- added C3: 100pF, rcl:C-USC0805
- added C4: 100nF, rcl:C-USC0805
- added D1: DB2S311, adafruit:DIODESOD-523
- added Q3: BSS138, SparkFun-DiscreteSemi:MOSFET-NCHANNELBSS138
- added R1: 1k, rcl:R-US_R0805
- added R7: 10k, rcl:R-US_R0805
- added U3: 74HCT1G125GW, NXP_By_element14_Batch_1:74HCT1G125GW
- C18: device rcl:C-USC0603 -> rcl:C-USC0805
Connections:
- removed net ESP_GPIO13_3V3: MDL1.GPIO13
- removed net LED: J4.2
- removed net SCL: R16.1, U4.SCL
- removed net SDA: R17.1, U4.SDA
- new net LED/RX: MDL1.RXD, U3.A
- new net MISO: MDL1.GPIO12, U2.SO
- new net MOSI: MDL1.GPIO13, U2.SI
- new net N$11: J4.2, U3.Y
- new net N$4: R7.2, U3.~OE
- new net N$7: BAT2.+, D1.A
- new net N$8: D1.C, R1.2
- new net RTC_!CS: U2.!CS
- new net SCK: MDL1.GPIO14, U2.SCK
- new net TX: MDL1.TXD
- net +3V3: now also C18.1, R14.2, U2.VCC
- net +5V: now also C4.1, U3.VCC; no longer C18.1, R14.2, R16.2, R17.2, U4.VCC
- net BOTON: no longer MDL1.GPIO14
- net ESP_RX_3V3: no longer MDL1.RXD
- net ESP_TX_3V3: no longer MDL1.TXD
- net GND: now also BAT2.-, C1.2, C2.2, C3.2, C4.2, R7.1, U2.VSS, U3.GND; no longer BT1.V-, U4.GND
- net N$2: now also C1.1, U2.X1, Y1.2; no longer U4.X1, Y2.2
- net N$3: now also C2.1, U2.X2, Y1.1; no longer U4.X2, Y2.1
- net N$6: now also U2.MFP; no longer U4.SQW
- net N$9: now also C3.1, R1.1, U2.VBAT; no longer BT1.V+, U4.VBATT
Other:
- moved on the sheet: C1, C13, C14, C16, C18, J2, J4, R14, U1, U2, Y1

Commit message: esquematico y bom v3 completo
Parts:
- removed BAT2: BAT-HLD-001, battery:LINX-BAT-HLD-00120SMD
- removed C14: 1200uF, rcl:CPOL-USUD-10X10
- removed C16: 10uF, rcl:CPOL-USUD-5X5,8
- removed C17: 1uF, rcl:C-USC0805
- removed C18: 100nF, rcl:C-USC0805
- removed D2: CD1206-S01575, diode:DIODE-MINIMELF
- removed J5: HDMI, partes v2:HDMI
- removed J6: FEMALE 2x3, SparkFun-Connectors:M03X2FEMALE
- removed K1: (no value), pimoroni-mechanical:RELAY_EE2
- removed Q2: PMBT3904, diego:PMBT3904
- removed Q3: BSS138, SparkFun-DiscreteSemi:MOSFET-NCHANNELBSS138
- removed R15: 10k, rcl:R-US_R0603
- added BAT1: BAT-HLD-001, battery:LINX-BAT-HLD-00120SMD
- added C11: 1200uF, rcl:CPOL-USUD-10X10
- added C12: 10uF, rcl:C-USC0805
- added C5: 100nF, rcl:C-USC0805
- added J1: JST-3, partes v2:JST-3
- added JP1: (no value), SparkFun-Connectors:M081X08
- added R10, R8: 10k, rcl:R-US_R0805
- added R11: 1k, rcl:R-US_R0805
- added U4: 74HCT1G125GW, NXP_By_element14_Batch_1:74HCT1G125GW
- added U5: NCP1117LPST33T3G, SparkFun-PowerIC:V_REG_LM1117SOT223
- C1: value 18pF -> 100nF
- C10: device rcl:C-USC0603 -> rcl:C-USC0805
- C2: value 18pF -> 100pF
- C3: value 100pF -> 18pF
- C4: value 100nF -> 18pF
- C6: value 470pF -> 100uF; device rcl:C-USC0603 -> rcl:C-USC1206
- C7: value 100uF -> 100nF; device rcl:C-USC1206 -> rcl:C-USC0805
- C8: value 10uF -> 100nF
- C9: value 1uF -> 100nF
- J2: value 1981584-1 -> HDMI; device con-usb:1981584-1 -> partes v2:HDMI
- J4: value JST-3 -> 1981584-1; device partes v2:JST-3 -> con-usb:1981584-1
- R1, R13, R9: value 1k -> 10k
- R14: value 10k -> 27k; device rcl:R-US_R0603 -> rcl:R-US_R0805
- R2, R3, R4, R6: device rcl:R-US_R0603 -> rcl:R-US_R0805
- R5: value 10k -> 1k; device rcl:R-US_R0603 -> rcl:R-US_R0805
- U1: value NCP1117LPST33T3G -> 74HCT1G125GW; device SparkFun-PowerIC:V_REG_LM1117SOT223 -> NXP_By_element14_Batch_1:74HCT1G125GW
- U3: value 74HCT1G125GW -> MC74VHC1GT66; device NXP_By_element14_Batch_1:74HCT1G125GW -> hoky:MC74VHC1GT66
Connections:
- removed net ESP_OC_NPROG: J6.5, MDL1.GPIO0, R2.1
- removed net ESP_OC_NRST: C6.1, J6.4, MDL1.REST, R6.1
- removed net ESP_RX_3V3: J6.1
- removed net ESP_TX_3V3: J6.2
- removed net HDMI_A_5V: J3.+5V, K1.MAIN1
- removed net HDMI_B_5V: J5.+5V, K1.OFF1
- removed net LVLSHF_OC_OE: J6.3
- removed net N$13: MDL1.GPIO2, R4.1
- removed net N$20: Q1.B, R9.2
- removed net RELE: R9.1
- removed net RFID_MISO_3V3: A1.MISO
- removed net RFID_MOSI_3V3: A1.MOSI
- removed net RFID_OC_NRST: A1.RST
- removed net RFID_SCK_3V3: A1.SCK
- removed net RFID_SS_3V3: A1.SDA/SS
- removed net RST_ATM_3V3: MDL1.GPIO4
- removed net RTC_!CS: U2.!CS
- new net !RST: C5.1, JP1.6, MDL1.REST, R7.1
- new net HDMI_IN_5V: J2.+5V, MDL1.GPIO5, R9.2, U3.P$1
- new net HDMI_OUT_5V: J3.+5V, JP1.1, U3.P$2, U4.Y
- new net HDMI_SW: MDL1.GPIO15, R2.2, U3.P$4, U4.A
- new net PROG/RTC_!CS: JP1.7, MDL1.GPIO0, R1.1, U2.!CS
- new net RFID_!CS: A1.SDA/SS, MDL1.GPIO2, R3.1
- net +3V3: now also C13.1, C6.1, JP1.3, R1.2, R3.2, R7.2, R8.2, S1.P$1, U5.OUT, U5.OUT@1; no longer C10.1, C16.+, C18.1, C8.1, C9.1, R14.2, R15.2, R2.2, R4.2, R5.2, U1.OUT, U1.OUT@1
- net +5V: now also C1.1, C10.1, C11.+, C12.1, C8.1, C9.1, J1.3, J4.VBUS, JP1.2, R12.2, U1.VCC, U3.P$5, U4.VCC, U5.IN; no longer C13.1, C14.+, C17.1, C4.1, D2.C, J2.VBUS, J4.3, K1.COIL+, R13.2, U1.IN, U3.VCC
- net BOTON: now also MDL1.ADC, R13.2, R14.1; no longer R15.1, S1.P$1
- net BUZZER: now also MDL1.GPIO4, R11.1; no longer R12.1
- net CLK_N: now also J2.CLK_N; no longer J5.CLK_N
- net CLK_P: now also J2.CLK_P; no longer J5.CLK_P
- net GND: now also BAT1.-, C11.-, C12.2, C5.2, J1.1, J2.GND@1, J2.GND@2, J2.GND@3, J2.GND@4, J2.GND@5, J2.GND@6, J2.GND@7, J2.GND@8, J2.GND@9, J4.GND, J4.S1, J4.S2, J4.S3, J4.S4, JP1.8, R10.1, R13.1, R2.1, R4.1, R9.1, U1.GND, U3.P$3, U4.GND, U5.ADJ; no longer BAT2.-, C14.-, C16.-, C17.2, C18.2, J2.GND, J2.S1, J2.S2, J2.S3, J2.S4, J4.1, J5.GND@1, J5.GND@2, J5.GND@3, J5.GND@4, J5.GND@5, J5.GND@6, J5.GND@7, J5.GND@8, J5.GND@9, J6.6, Q2.E, R3.1, R7.1, S1.P$2, U1.ADJ, U3.GND
- net LED/RX: now also JP1.4, U1.A; no longer U3.A
- net MISO: now also A1.MISO
- net MOSI: now also A1.MOSI
- net N$1: now also Q1.B, R11.2; no longer Q2.B, R12.2
- net N$10: now also R6.1; no longer R5.1
- net N$11: now also J1.2, U1.Y; no longer J4.2, U3.Y
- net N$15: now also R10.2, U4.~OE; no longer D2.A, K1.COIL-, Q1.C
- net N$16: now also S1.P$2; no longer MDL1.GPIO15, R3.2
- net N$2: now also C3.1; no longer C1.1
- net N$3: now also C4.1; no longer C2.1
- net N$30: now also J2.CEC_DAT; no longer J5.CEC_DAT
- net N$31: now also J2.SCL; no longer J5.SCL
- net N$32: now also J2.SDA; no longer J5.SDA
- net N$33: now also J2.HPD; no longer J5.HPD
- net N$4: now also R4.2, U1.~OE; no longer R7.2, U3.~OE
- net N$5: now also Q1.C, R12.1; no longer Q2.C, R13.1
- net N$6: now also R8.1; no longer R14.1
- net N$7: now also BAT1.+; no longer BAT2.+
- net N$8: now also R5.2; no longer R1.2
- net N$9: now also C2.1, R5.1; no longer C3.1, R1.1
- net SCK: now also A1.SCK
- net TX: now also JP1.5
- net TX0_N: now also J2.TX0_N; no longer J5.TX0_N
- net TX0_P: now also J2.TX0_P; no longer J5.TX0_P
- net TX1_N: now also J2.TX1_N; no longer J5.TX1_N
- net TX1_P: now also J2.TX1_P; no longer J5.TX1_P
- net TX2_N: now also J2.TX2_N; no longer J5.TX2_N
- net TX2_P: now also J2.TX2_P; no longer J5.TX2_P
Other:
- note added: "Elegir uno"
- moved on the sheet: A1, C1, C10, C13, C2, C3, C4, C6, C7, C8, C9, D1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

Commit message: Ruteo pcb V3 completo
Parts:
- C11: value 1200uF -> 100uF; device rcl:CPOL-USUD-10X10 -> rcl:CPOL-USUD-6,3X5,8
- R13: value 10k -> 27k
- R14: value 27k -> 10k
Connections:
- removed net N$16: S1.P$2
- new net N$12: R13.2, S1.P$2
- net BOTON: now also R13.1, R14.2; no longer R13.2, R14.1
- net GND: now also JP1.1, R14.1; no longer JP1.8, R13.1
- net HDMI_OUT_5V: now also JP1.8; no longer JP1.1
- net N$2: now also Y1.1; no longer Y1.2
- net N$3: now also Y1.2; no longer Y1.1
Other:
- moved on the sheet: R13, R14, Y1
Changed lines of the file:
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@@
 <setting verticaltext="up"/>
 </settings>
-<grid distance="0.1" unitdist="inch" unit="inch" style="dots" multiple="1" display="yes" altdistance="0.01" altunitdist="inch" altunit="inch"/>
+<grid distance="0.1" unitdist="inch" unit="inch" style="lines" multiple="1" display="no" altdistance="0.01" altunitdist="inch" altunit="inch"/>
 <layers>
 <layer number="1" name="Top" color="4" fill="1" visible="no" active="no"/>
@@
 <part name="GND8" library="supply1" deviceset="GND" device=""/>
 <part name="J4" library="con-usb" deviceset="1981584-1" device=""/>
-<part name="C11" library="rcl" deviceset="CPOL-US" device="UD-10X10" value="1200uF"/>
 <part name="C13" library="rcl" deviceset="C-US" device="C0805" value="10uF"/>
 <part name="SP1" library="adafruit" deviceset="SPEAKER" device="/PS12"/>
@@
 <part name="C8" library="rcl" deviceset="C-US" device="C0805" value="100nF"/>
 <part name="GND15" library="supply1" deviceset="GND" device=""/>
-<part name="R13" library="rcl" deviceset="R-US_" device="R0805" value="10k"/>
+<part name="R14" library="rcl" deviceset="R-US_" device="R0805" value="10k"/>
 <part name="C12" library="rcl" deviceset="C-US" device="C0805" value="10uF"/>
 <part name="U4" library="NXP_By_element14_Batch_1" deviceset="74HCT1G125GW" device=""/>
@@
 <part name="+3V36" library="supply1" deviceset="+3V3" device=""/>
 <part name="GND22" library="supply1" deviceset="GND" device=""/>
-<part name="R14" library="rcl" deviceset="R-US_" device="R0805" value="27k"/>
+<part name="R13" library="rcl" deviceset="R-US_" device="R0805" value="27k"/>
+<part name="C11" library="rcl" deviceset="CPOL-US" device="UD-6,3X5,8" value="100uF"/>
 </parts>
 <sheets>
@@
 <instance part="GND8" gate="1" x="109.22" y="-12.7" rot="MR0"/>
 <instance part="J4" gate="G$1" x="314.96" y="-7.62" rot="MR0"/>
-<instance part="C11" gate="G$1" x="335.28" y="-7.62"/>
 <instance part="C13" gate="G$1" x="383.54" y="-10.16"/>
 <instance part="SP1" gate="S1" x="264.16" y="-2.54" smashed="yes" rot="R270">
@@
 </instance>
 <instance part="U2" gate="G$1" x="111.76" y="129.54"/>
-<instance part="Y1" gate="G$1" x="88.9" y="154.94" rot="R90"/>
+<instance part="Y1" gate="G$1" x="88.9" y="154.94" rot="R270"/>
 <instance part="C3" gate="G$1" x="78.74" y="160.02" rot="R270"/>
 <instance part="BAT1" gate="G$1" x="43.18" y="119.38" rot="R270"/>
@@
 <instance part="C8" gate="G$1" x="233.68" y="114.3" rot="R270"/>
 <instance part="GND15" gate="1" x="223.52" y="106.68"/>
-<instance part="R13" gate="G$1" x="342.9" y="88.9" rot="R90"/>
+<instance part="R14" gate="G$1" x="342.9" y="88.9" rot="R90"/>
 <instance part="C12" gate="G$1" x="347.98" y="-7.62"/>
 <instance part="U4" gate="A" x="264.16" y="48.26"/>
@@
 <instance part="GND14" gate="1" x="180.34" y="33.02"/>
 <instance part="JP1" gate="G$1" x="350.52" y="45.72" rot="R180"/>
-<instance part="P+7" gate="1" x="340.36" y="58.42"/>
-<instance part="+3V36" gate="G$1" x="332.74" y="58.42"/>
-<instance part="GND22" gate="1" x="340.36" y="27.94"/>
-<instance part="R14" gate="G$1" x="342.9" y="104.14" rot="R90"/>
+<instance part="P+7" gate="1" x="340.36" y="60.96"/>
+<instance part="+3V36" gate="G$1" x="332.74" y="60.96"/>
+<instance part="GND22" gate="1" x="325.12" y="45.72"/>
+<instance part="R13" gate="G$1" x="342.9" y="104.14" rot="R90"/>
+<instance part="C11" gate="G$1" x="335.28" y="-7.62"/>
 </instances>
 <busses>
@@
 </segment>
 <segment>
-<wire x1="335.28" y1="-12.7" x2="335.28" y2="-15.24" width="0.1524" layer="91"/>
 <pinref part="GND24" gate="1" pin="GND"/>
+<wire x1="325.12" y1="-15.24" x2="335.28" y2="-15.24" width="0.1524" layer="91"/>
 <wire x1="335.28" y1="-15.24" x2="347.98" y2="-15.24" width="0.1524" layer="91"/>
 <wire x1="347.98" y1="-15.24" x2="347.98" y2="-17.78" width="0.1524" layer="91"/>
-<wire x1="325.12" y1="-15.24" x2="335.28" y2="-15.24" width="0.1524" layer="91"/>
-<junction x="335.28" y="-15.24"/>
 <wire x1="322.58" y1="-12.7" x2="325.12" y2="-12.7" width="0.1524" layer="91"/>
 <wire x1="325.12" y1="-12.7" x2="325.12" y2="-15.24" width="0.1524" layer="91"/>
@@
 <pinref part="J4" gate="G$1" pin="S4"/>
 <pinref part="J4" gate="G$1" pin="GND"/>
-<pinref part="C11" gate="G$1" pin="-"/>
 <pinref part="U5" gate="G$1" pin="ADJ"/>
 <wire x1="347.98" y1="-15.24" x2="360.68" y2="-15.24" width="0.1524" layer="91"/>
@@
 <pinref part="C12" gate="G$1" pin="2"/>
 <wire x1="347.98" y1="-12.7" x2="347.98" y2="-15.24" width="0.1524" layer="91"/>
+<pinref part="C11" gate="G$1" pin="-"/>
+<wire x1="335.28" y1="-12.7" x2="335.28" y2="-15.24" width="0.1524" layer="91"/>
+<junction x="335.28" y="-15.24"/>
 </segment>
 <segment>
@@
 <pinref part="GND23" gate="1" pin="GND"/>
 <wire x1="342.9" y1="83.82" x2="342.9" y2="81.28" width="0.1524" layer="91"/>
-<pinref part="R13" gate="G$1" pin="1"/>
+<pinref part="R14" gate="G$1" pin="1"/>
 </segment>
 <segment>
@@
 </segment>
 <segment>
-<pinref part="JP1" gate="G$1" pin="8"/>
 <pinref part="GND22" gate="1" pin="GND"/>
-<wire x1="345.44" y1="35.56" x2="340.36" y2="35.56" width="0.1524" layer="91"/>
-<wire x1="340.36" y1="35.56" x2="340.36" y2="30.48" width="0.1524" layer="91"/>
+<wire x1="325.12" y1="48.26" x2="325.12" y2="53.34" width="0.1524" layer="91"/>
+<pinref part="JP1" gate="G$1" pin="1"/>
+<wire x1="325.12" y1="53.34" x2="345.44" y2="53.34" width="0.1524" layer="91"/>
 </segment>
 </net>
@@
 <wire x1="335.28" y1="-2.54" x2="347.98" y2="-2.54" width="0.1524" layer="91"/>
 <wire x1="347.98" y1="-2.54" x2="353.06" y2="-2.54" width="0.1524" layer="91"/>
-<wire x1="335.28" y1="-5.08" x2="335.28" y2="-2.54" width="0.1524" layer="91"/>
 <junction x="335.28" y="-2.54"/>
 <pinref part="P+6" gate="1" pin="+5V"/>
@@
 <wire x1="335.28" y1="-2.54" x2="322.58" y2="-2.54" width="0.1524" layer="91"/>
 <pinref part="J4" gate="G$1" pin="VBUS"/>
-<pinref part="C11" gate="G$1" pin="+"/>
 <pinref part="U5" gate="G$1" pin="IN"/>
 <pinref part="C12" gate="G$1" pin="1"/>
 <wire x1="347.98" y1="-5.08" x2="347.98" y2="-2.54" width="0.1524" layer="91"/>
 <junction x="347.98" y="-2.54"/>
+<pinref part="C11" gate="G$1" pin="+"/>
+<wire x1="335.28" y1="-5.08" x2="335.28" y2="-2.54" width="0.1524" layer="91"/>
 </segment>
 <segment>
@@
 <segment>
 <pinref part="P+7" gate="1" pin="+5V"/>
-<wire x1="340.36" y1="55.88" x2="340.36" y2="50.8" width="0.1524" layer="91"/>
+<wire x1="340.36" y1="58.42" x2="340.36" y2="50.8" width="0.1524" layer="91"/>
 <pinref part="JP1" gate="G$1" pin="2"/>
 <wire x1="340.36" y1="50.8" x2="345.44" y2="50.8" width="0.1524" layer="91"/>
@@
 <pinref part="+3V36" gate="G$1" pin="+3V3"/>
 <wire x1="345.44" y1="48.26" x2="332.74" y2="48.26" width="0.1524" layer="91"/>
-<wire x1="332.74" y1="48.26" x2="332.74" y2="55.88" width="0.1524" layer="91"/>
+<wire x1="332.74" y1="48.26" x2="332.74" y2="58.42" width="0.1524" layer="91"/>
 </segment>
 </net>
@@
 <pinref part="U4" gate="A" pin="Y"/>
 <wire x1="281.94" y1="50.8" x2="294.64" y2="50.8" width="0.1524" layer="91"/>
-<wire x1="294.64" y1="50.8" x2="294.64" y2="66.04" width="0.1524" layer="91"/>
 <junction x="294.64" y="101.6"/>
-<pinref part="JP1" gate="G$1" pin="1"/>
-<wire x1="294.64" y1="66.04" x2="294.64" y2="101.6" width="0.1524" layer="91"/>
-<wire x1="345.44" y1="53.34" x2="342.9" y2="53.34" width="0.1524" layer="91"/>
-<wire x1="342.9" y1="53.34" x2="342.9" y2="66.04" width="0.1524" layer="91"/>
-<wire x1="342.9" y1="66.04" x2="294.64" y2="66.04" width="0.1524" layer="91"/>
-<junction x="294.64" y="66.04"/>
+<wire x1="294.64" y1="50.8" x2="294.64" y2="101.6" width="0.1524" layer="91"/>
+<pinref part="JP1" gate="G$1" pin="8"/>
+<wire x1="345.44" y1="35.56" x2="294.64" y2="35.56" width="0.1524" layer="91"/>
+<wire x1="294.64" y1="35.56" x2="294.64" y2="50.8" width="0.1524" layer="91"/>
+<junction x="294.64" y="50.8"/>
 </segment>
 </net>
@@
 <junction x="342.9" y="96.52"/>
 <label x="335.28" y="96.52" size="1.27" layer="95" rot="R180" xref="yes"/>
-<pinref part="R13" gate="G$1" pin="2"/>
-<pinref part="R14" gate="G$1" pin="1"/>
+<pinref part="R14" gate="G$1" pin="2"/>
+<pinref part="R13" gate="G$1" pin="1"/>
 </segment>
 </net>
@@
 <segment>
 <pinref part="C3" gate="G$1" pin="1"/>
-<pinref part="Y1" gate="G$1" pin="2"/>
 <wire x1="81.28" y1="160.02" x2="88.9" y2="160.02" width="0.1524" layer="91"/>
-<wire x1="88.9" y1="160.02" x2="88.9" y2="157.48" width="0.1524" layer="91"/>
+<pinref part="U2" gate="G$1" pin="X1"/>
 <wire x1="88.9" y1="160.02" x2="96.52" y2="160.02" width="0.1524" layer="91"/>
-<junction x="88.9" y="160.02"/>
-<pinref part="U2" gate="G$1" pin="X1"/>
 <wire x1="99.06" y1="134.62" x2="96.52" y2="134.62" width="0.1524" layer="91"/>
 <wire x1="96.52" y1="134.62" x2="96.52" y2="160.02" width="0.1524" layer="91"/>
+<pinref part="Y1" gate="G$1" pin="1"/>
+<wire x1="88.9" y1="157.48" x2="88.9" y2="160.02" width="0.1524" layer="91"/>
+<junction x="88.9" y="160.02"/>
 </segment>
 </net>
 <net name="N$3" class="0">
 <segment>
-<pinref part="Y1" gate="G$1" pin="1"/>
-<wire x1="88.9" y1="152.4" x2="88.9" y2="149.86" width="0.1524" layer="91"/>
 <pinref part="C4" gate="G$1" pin="1"/>
 <wire x1="88.9" y1="149.86" x2="81.28" y2="149.86" width="0.1524" layer="91"/>
-<junction x="88.9" y="149.86"/>
 <pinref part="U2" gate="G$1" pin="X2"/>
 <wire x1="88.9" y1="149.86" x2="88.9" y2="132.08" width="0.1524" layer="91"/>
 <wire x1="88.9" y1="132.08" x2="99.06" y2="132.08" width="0.1524" layer="91"/>
+<pinref part="Y1" gate="G$1" pin="2"/>
+<wire x1="88.9" y1="152.4" x2="88.9" y2="149.86" width="0.1524" layer="91"/>
+<junction x="88.9" y="149.86"/>
 </segment>
 </net>
@@
 </segment>
 </net>
-<net name="N$16" class="0">
+<net name="N$12" class="0">
 <segment>
 <pinref part="S1" gate="G$1" pin="P$2"/>
+<pinref part="R13" gate="G$1" pin="2"/>
 <wire x1="342.9" y1="111.76" x2="342.9" y2="109.22" width="0.1524" layer="91"/>
 </segment>

Commit message: gerbers v3
Parts:
- added R15, R16: 10k, rcl:R-US_R0805
- C11: device rcl:CPOL-USUD-6,3X5,8 -> hoky:CPOL-US
- R13: value 27k -> 10k
Connections:
- new net N$13: R13.1, R15.2
- new net N$14: R15.1, R16.2
- net BOTON: now also R16.1; no longer R13.1
Other:
- moved on the sheet: R13, R14, S1
Changed lines of the file:
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@@
 <part name="+3V36" library="supply1" deviceset="+3V3" device=""/>
 <part name="GND22" library="supply1" deviceset="GND" device=""/>
-<part name="R13" library="rcl" deviceset="R-US_" device="R0805" value="27k"/>
-<part name="C11" library="rcl" deviceset="CPOL-US" device="UD-6,3X5,8" value="100uF"/>
+<part name="R13" library="rcl" deviceset="R-US_" device="R0805" value="10k"/>
+<part name="C11" library="hoky" deviceset="CPOL-US" device="" value="100uF"/>
+<part name="R15" library="rcl" deviceset="R-US_" device="R0805" value="10k"/>
+<part name="R16" library="rcl" deviceset="R-US_" device="R0805" value="10k"/>
 </parts>
 <sheets>
@@
 <instance part="GND13" gate="1" x="180.34" y="149.86"/>
 <instance part="GND21" gate="1" x="292.1" y="149.86"/>
-<instance part="S1" gate="G$1" x="342.9" y="116.84" smashed="yes" rot="R270">
-<attribute name="NAME" x="345.44" y="119.38" size="1.778" layer="95"/>
-<attribute name="VALUE" x="345.44" y="121.92" size="1.778" layer="96"/>
+<instance part="S1" gate="G$1" x="342.9" y="137.16" smashed="yes" rot="R270">
+<attribute name="NAME" x="345.44" y="139.7" size="1.778" layer="95"/>
+<attribute name="VALUE" x="345.44" y="142.24" size="1.778" layer="96"/>
 </instance>
-<instance part="GND23" gate="1" x="342.9" y="78.74"/>
+<instance part="GND23" gate="1" x="342.9" y="73.66"/>
 <instance part="P+2" gate="1" x="109.22" y="7.62" rot="MR0"/>
 <instance part="GND8" gate="1" x="109.22" y="-12.7" rot="MR0"/>
@@
 <instance part="+3V35" gate="G$1" x="160.02" y="-2.54"/>
 <instance part="GND12" gate="1" x="162.56" y="-22.86"/>
-<instance part="+3V37" gate="G$1" x="342.9" y="129.54"/>
+<instance part="+3V37" gate="G$1" x="342.9" y="149.86"/>
 <instance part="U5" gate="G$1" x="360.68" y="-2.54" smashed="yes">
 <attribute name="NAME" x="363.22" y="-10.16" size="1.778" layer="95"/>
@@
 <instance part="C8" gate="G$1" x="233.68" y="114.3" rot="R270"/>
 <instance part="GND15" gate="1" x="223.52" y="106.68"/>
-<instance part="R14" gate="G$1" x="342.9" y="88.9" rot="R90"/>
+<instance part="R14" gate="G$1" x="342.9" y="83.82" rot="R90"/>
 <instance part="C12" gate="G$1" x="347.98" y="-7.62"/>
 <instance part="U4" gate="A" x="264.16" y="48.26"/>
@@
 <instance part="+3V36" gate="G$1" x="332.74" y="60.96"/>
 <instance part="GND22" gate="1" x="325.12" y="45.72"/>
-<instance part="R13" gate="G$1" x="342.9" y="104.14" rot="R90"/>
+<instance part="R13" gate="G$1" x="342.9" y="124.46" rot="R90"/>
 <instance part="C11" gate="G$1" x="335.28" y="-7.62"/>
+<instance part="R15" gate="G$1" x="342.9" y="111.76" rot="R90"/>
+<instance part="R16" gate="G$1" x="342.9" y="99.06" rot="R90"/>
 </instances>
 <busses>
@@
 <segment>
 <pinref part="GND23" gate="1" pin="GND"/>
-<wire x1="342.9" y1="83.82" x2="342.9" y2="81.28" width="0.1524" layer="91"/>
+<wire x1="342.9" y1="78.74" x2="342.9" y2="76.2" width="0.1524" layer="91"/>
 <pinref part="R14" gate="G$1" pin="1"/>
 </segment>
@@
 <pinref part="+3V37" gate="G$1" pin="+3V3"/>
 <pinref part="S1" gate="G$1" pin="P$1"/>
-<wire x1="342.9" y1="127" x2="342.9" y2="121.92" width="0.1524" layer="91"/>
+<wire x1="342.9" y1="147.32" x2="342.9" y2="142.24" width="0.1524" layer="91"/>
 </segment>
 <segment>
@@
 </segment>
 <segment>
-<wire x1="342.9" y1="99.06" x2="342.9" y2="96.52" width="0.1524" layer="91"/>
-<wire x1="342.9" y1="96.52" x2="342.9" y2="93.98" width="0.1524" layer="91"/>
-<wire x1="342.9" y1="96.52" x2="335.28" y2="96.52" width="0.1524" layer="91"/>
-<junction x="342.9" y="96.52"/>
-<label x="335.28" y="96.52" size="1.27" layer="95" rot="R180" xref="yes"/>
+<wire x1="342.9" y1="91.44" x2="342.9" y2="88.9" width="0.1524" layer="91"/>
+<wire x1="342.9" y1="91.44" x2="335.28" y2="91.44" width="0.1524" layer="91"/>
+<label x="335.28" y="91.44" size="1.27" layer="95" rot="R180" xref="yes"/>
 <pinref part="R14" gate="G$1" pin="2"/>
-<pinref part="R13" gate="G$1" pin="1"/>
+<pinref part="R16" gate="G$1" pin="1"/>
+<wire x1="342.9" y1="93.98" x2="342.9" y2="91.44" width="0.1524" layer="91"/>
+<junction x="342.9" y="91.44"/>
 </segment>
 </net>
@@
 <pinref part="S1" gate="G$1" pin="P$2"/>
 <pinref part="R13" gate="G$1" pin="2"/>
-<wire x1="342.9" y1="111.76" x2="342.9" y2="109.22" width="0.1524" layer="91"/>
-</segment>
-</net>
+<wire x1="342.9" y1="132.08" x2="342.9" y2="129.54" width="0.1524" layer="91"/>
+</segment>
+</net>
+<net name="N$13" class="0">
+<segment>
+<pinref part="R13" gate="G$1" pin="1"/>
+<pinref part="R15" gate="G$1" pin="2"/>
+<wire x1="342.9" y1="119.38" x2="342.9" y2="116.84" width="0.1524" layer="91"/>
+</segment>
+</net>
+<net name="N$14" class="0">
+<segment>
+<pinref part="R15" gate="G$1" pin="1"/>
+<pinref part="R16" gate="G$1" pin="2"/>
+<wire x1="342.9" y1="106.68" x2="342.9" y2="104.14" width="0.1524" layer="91"/>
+</segment>
+</net>
